File: hardware/fpga.sch (KiCad schematic (older format))
At the start: 68 parts, among them J2 ETHERNET_DUAL, P1 CONN_01X03, P2 CONN_01X03, P3 CONN_01X03, P4 CONN_01X03, P5 CONN_02X07, U2 XC6SLXN-TQG144, U3 W25Q80DV, U4 KSZ9031RNXCA, U6 511FBA125M000BAG, U7 KSZ9031RNXCA

Commit message: Backup, clearing bottom of power section.
Connections:
- wire segments 467 -> 443
Other:
- moved on the sheet: J2B

Commit message: Progress.
Parts:
- added C33, C60: 100nF, 00_Passives:C0603, symbol C
- added D2: LED_592, 00_Passives:LED_592-3030-013F, symbol LED_592
- added D5: DIODE, Diodes_SMD:SOD-323, symbol DIODE
- added M13: BSS138, 00_Passives:SOT23_GSD, symbol NMOS
- added P25, P26: CONN_01X03, Pin_Headers:Pin_Header_Straight_1x03, symbol CONN_01X03
- added P27, P28, P29, P30: CONN_01X02, Connect:PINHEAD1-2, symbol CONN_01X02
- added R131, R132, R133, R134: 220, 00_Passives:R0603, symbol R
- added U57: LM75, Housings_SOIC:SOIC-8_3.9x4.9mm_Pitch1.27mm, symbol LM75
- added U60: UCN5841A, Housings_DIP:DIP-18_W7.62mm, symbol UCN5841A
- added U61: DS28CM00, 00_Passives:SOT23_5, symbol DS28CM00
Connections:
- net labels added: +12V, AUX_CLK, AUX_DATA, AUX_STR, FAN, SCL, SDA
- wire segments 443 -> 527
Other:
- note added: "A6841 is alternatief (op voorraad)"
- moved on the sheet: C1, C10, C11, C12, C13, C14, C15, C16, C17, C18, C2, C3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

Commit message: Backup
Parts:
- added C132, C133, C134, C135, C136, C137, C138, C139, C140, C141, C142, C143, C144, C145, C146, C147, C148, C149, C150, C151, C152, C153, C154: 100nF, 00_Passives:C0603, symbol C
- added R139: 1.0k, 00_Passives:R0603, symbol R
Connections:
- net labels removed: HB_DISABLE
- wire segments 527 -> 592
