File: hardware/drive.sch (KiCad schematic (older format))
At the start: 112 parts, among them J1 DB25_STACKED, M1 NMOS, M2 NMOS, M3 NMOS, M4 NMOS, M5 NMOS, M6 NMOS, P11 CONN_01X01, P12 CONN_01X01, P15 CONN_01X01, P17 CONN_01X01, P19 CONN_01X01, P20 CONN_01X01, P23 CONN_01X01, P24 CONN_01X01, P6 CONN_01X01, U10 MAX3463, U11 MAX3463, U12 MAX3463, U13 MAX3463, U14 MAX3463, U15 ADuM3223BRZ, U16 TS321, U17 ACS758, U18 ADuM3223BRZ, U19 AD8226, U20 AD8226, U21 AD8226, U24 ACS758, U25 AMC1204, U42 LT3010, U47 TS321, U49 TS321, U8 ADuM3223BRZ, U9 ACS758, X1 NMK1212SAC

Commit message: Backup, clearing bottom of power section.
Parts:
- removed C24, C25, C29, C30: 1uF, 00_Local:C0805, symbol C
- removed C37: 1uF/630V, Capacitors_SMD:C_2220, symbol C
- removed C38: 100uF/16V, Capacitors_SMD:c_elec_6.3x5.3, symbol CAPAPOL
- removed D2, D3, D5, D6: S1M, 00_Passives:DO-214AC(SMA), symbol DIODE
- removed M1, M2, M3, M4, M5, M6: NMOS, 00_Passives:TO-247_GDS_below_board, symbol NMOS
- removed P19, P24: CONN_01X01, 00_Passives:conn_01x01_3mm, symbol CONN_01X01
- removed R101, R99: 10k, 00_Passives:R0603, symbol R
- removed R24: 22, 00_Local:R0603, symbol R
- removed R30, R44: 2k, 00_Local:R0603, symbol R
- removed R36: 22, 00_Local:R0805, symbol R
- removed R51: 51, 00_Local:R0603, symbol R
- removed U15, U18, U8: ADuM3223BRZ, Housings_SOIC:SOIC-16_3.9x9.9mm_Pitch1.27mm, symbol ADuM3223BRZ
- removed U17, U24, U9: ACS758, 00_Passives:acs758, symbol ACS758
- removed U47, U49: TS321, 00_Passives:SOT23_5, symbol TS321
- added C113, C50, C52, C56: 1uF, 00_Local:C0805, symbol C
- added C115, C116, C119, C120, C123, C125: 100nF, 00_Passives:C0603, symbol C
- added C57: 1uF/630V, Capacitors_SMD:C_2220, symbol C
- added C64: 10nF, 00_Passives:C0603, symbol C
- added C65: 10uF, 00_Passives:C1210, symbol C
- added D10: S1M, 00_Passives:DO-214AC(SMA), symbol DIODE
- added M1, M10, M12, M3, M5, M8: C3M0280090J, 00_Passives:TO-263-7-GDSKS, symbol NMOS_KELVIN
- added P18, P9: CONN_01X01, 00_Passives:conn_01x01_3mm, symbol CONN_01X01
- added R100: 220, 00_Passives:R0603, symbol R
- added R102, R127: 51, 00_Local:R0603, symbol R
- added R113, R61: 22, 00_Local:R0603, symbol R
- added R115, R117, R67, R72: 10k, 00_Passives:R0603, symbol R
- added R120, R81: 2k, 00_Local:R0603, symbol R
- added R121, R126: R, 00_Local:R0603, symbol R
- added R123, R87: 1k, 00_Local:R0603, symbol R
- added R129: 0.1, 00_Local:R0603, symbol R
- added U17, U24, U34, U49, U51, U8: Si8261BCD-C-IS, 00_Passives:SOIC-6_6.8x4.6mm_Pitch1.27mm, symbol Si8261BCD-C-IS
- added U43, U54, U9: ACS722KMATR-20AB-T, Housings_SOIC:SOIC-16_7.5x10.3mm_Pitch1.27mm, symbol ACS722KMATR-20AB-T
- added U46, U55: TS321, 00_Passives:SOT23_5, symbol TS321
- C27: value 1uF/630V -> 1uF; footprint Capacitors_SMD:C_2220 -> 00_Local:C0805
- C32: value 47pF -> 1uF/630V; footprint 00_Local:C0603 -> Capacitors_SMD:C_2220
- C41: value 47pF -> 10nF; footprint 00_Local:C0603 -> 00_Passives:C0603
- C45, C67: value 10nF -> 47pF; footprint 00_Passives:C0603 -> 00_Local:C0603
- P6: Farnell (none) -> 2497613
- R103: value 10k -> 22; footprint 00_Passives:R0603 -> 00_Local:R0603
- R16: footprint 00_Local:R0805 -> 00_Local:R0603
- R25: value 22 -> 220; footprint 00_Local:R0805 -> 00_Passives:R0603
- R34: value 1k -> 220; footprint 00_Local:R0603 -> 00_Passives:R0603
- R35: value 22 -> 220; footprint 00_Local:R0603 -> 00_Passives:R0603
- R37: value 51 -> 220; footprint 00_Local:R0603 -> 00_Passives:R0603
- R50: value 1k -> 22
- R98: value 10k -> 220
- X1: value NMK1212SAC -> RKZ1215S
Connections:
- net labels added: HB0, HB1, HB2, HV0, HV1, HV2, ISOL_15V, OUT0, OUT1, OUT2
- net labels removed: DISABLE, ISOL_12V
- wire segments 417 -> 467
Other:
- moved on the sheet: C20, C22, C26, C33, C34, C35, C36, C39, C43, C73, J1A, P11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

Commit message: Progress.
Parts:
- removed C33: 100uF/16V, Capacitors_SMD:c_elec_6.3x5.3, symbol CAPAPOL
- removed X1: RKZ1215S, 00_Passives:RKZXXXXS, symbol NMK1212SAC
- added C127, C129, C130: 100nF, 00_Passives:C0603, symbol C
- added R135: 15k, 00_Passives:R0603, symbol R
- added R138: 4.7k, 00_Passives:R0603, symbol R
- added U58: ips511g, Housings_SOIC:SOIC-8_3.9x4.9mm_Pitch1.27mm, symbol ips511g
- added X1: R2S-1215/H, 00_Passives:RECOM_R2S, symbol R2S-xxxx
- P11, P12, P15, P17, P18, P20, P23, P6, P9: footprint 00_Passives:conn_01x01_3mm -> 00_Passives:WE_9774080151R
Connections:
- net +12V: now also U58.5 (Vcc), U58.6 (Vcc), U58.7 (Vcc), U58.8 (Vcc), X1.2 (vip)
- net +3.3V: now also C127.1, C129.1, C130.1
- net +5V: now also J1.B21 (21), J1.B8 (8), J1.B9 (9), R135.2, R138.2; no longer J1.A21 (21), J1.A8 (8), J1.A9 (9)
- net AN0_N: now also J1.B25 (P25); no longer J1.A25 (P25)
- net AN0_P: now also J1.B13 (13); no longer J1.A13 (13)
- net AN1_N: now also J1.B24 (A24); no longer J1.A24
- net AN1_P: now also J1.B12 (12); no longer J1.A12 (12)
- net AN2_N: now also J1.B23 (P23); no longer J1.A23 (P23)
- net AN2_P: now also J1.B11 (11); no longer J1.A11 (11)
- net BRIDGE-: now also X1.4 (von)
- net ENC0_N: now also J1.B5 (5); no longer J1.A5 (5)
- net ENC0_P: now also J1.B18 (P18); no longer J1.A18 (P18)
- net ENC1_N: now also J1.B4 (4); no longer J1.A4 (4)
- net ENC1_P: now also J1.B17 (17); no longer J1.A17 (17)
- net ENC2_N: now also J1.B3 (3); no longer J1.A3 (3)
- net ENC2_P: now also J1.B16 (A16); no longer J1.A16
- net ENC3_N: now also J1.B2 (A2); no longer J1.A2
- net ENC3_P: now also J1.B15 (P15); no longer J1.A15 (P15)
- net ENC4_N: now also J1.B1 (1); no longer J1.A1 (1)
- net ENC4_P: now also J1.B14 (P14); no longer J1.A14 (P14)
- net GND: now also J1.B10 (10), J1.B19 (P19), J1.B22 (P22), J1.B6 (6), C127.2, C129.2, C130.2, U58.1 (GND), X1.1 (vin); no longer J1.A10 (10), J1.A19 (P19), J1.A22 (P22), J1.A6 (6)
- net ISOL_15V: now also X1.5 (vop)
- new net: J1.B20 (P20), J1.B7 (7), U58.4 (OUT)
- new net: R138.1, U58.2 (IN)
- new net: R135.1, U58.3 (DG)

Commit message: Backup
Parts:
- removed C116, C120, C125: 100nF, 00_Passives:C0603, symbol C
Connections:
- net -5V is gone; now on net GND: U16.2 (V-), U46.2 (V-), U55.2 (V-)

Commit message: First small drive hardware.
Parts:
- R115, R67, R93: Imax (none) -> 1.65e-4
- U16, U46, U55: Imax_5 (none) -> 3e-3
- U25: Imax_1 (none) -> 16e-3; Imax_8 (none) -> 4e-3
- U43, U54, U9: Imax_10 (none) -> 12e-3
Connections:
- net +5V: now also J1.A21 (21), J1.A8 (8), J1.A9 (9); no longer J1.B21 (21), J1.B8 (8), J1.B9 (9)
- net AN0_N: now also J1.A25 (P25); no longer J1.B25 (P25)
- net AN0_P: now also J1.A13 (13); no longer J1.B13 (13)
- net AN1_N: now also J1.A24; no longer J1.B24 (A24)
- net AN1_P: now also J1.A12 (12); no longer J1.B12 (12)
- net AN2_N: now also J1.A23 (P23); no longer J1.B23 (P23)
- net AN2_P: now also J1.A11 (11); no longer J1.B11 (11)
- net ENC0_N: now also J1.A5 (5); no longer J1.B5 (5)
- net ENC0_P: now also J1.A18 (P18); no longer J1.B18 (P18)
- net ENC1_N: now also J1.A4 (4); no longer J1.B4 (4)
- net ENC1_P: now also J1.A17 (17); no longer J1.B17 (17)
- net ENC2_N: now also J1.A3 (3); no longer J1.B3 (3)
- net ENC2_P: now also J1.A16; no longer J1.B16 (A16)
- net ENC3_N: now also J1.A2; no longer J1.B2 (A2)
- net ENC3_P: now also J1.A15 (P15); no longer J1.B15 (P15)
- net ENC4_N: now also J1.A1 (1); no longer J1.B1 (1)
- net ENC4_P: now also J1.A14 (P14); no longer J1.B14 (P14)
- net GND: now also J1.A10 (10), J1.A19 (P19), J1.A22 (P22), J1.A6 (6); no longer J1.B10 (10), J1.B19 (P19), J1.B22 (P22), J1.B6 (6)
- new net: J1.A20 (P20), J1.A7 (7), U58.4 (OUT)
