File: hardware/motor_sturing.kicad_pcb (KiCad board)
At the start: 4 copper layers, 220 x 100 mm, 390 parts, among them J1 DB25_STACKED, J2 ETHERNET_DUAL, M1 C3M0280090J, M10 C3M0280090J, M11 C3M0280090J, M12 C3M0280090J, M13 BSS138, M2 C3M0280090J, M3 C3M0280090J, M4 C3M0280090J, M5 C3M0280090J, M6 C3M0280090J, M7 C3M0280090J, M8 C3M0280090J, M9 C3M0280090J, P1 CONN_01X03, P10 CONN_01X01, P11 CONN_01X01, P12 CONN_01X01, P13 CONN_01X01, P14 CONN_01X01, P15 CONN_01X01, P16 CONN_01X01, P17 CONN_01X01, P18 CONN_01X01, P19 CONN_01X01, P2 CONN_01X03, P20 CONN_01X01, P21 CONN_01X01, P22 CONN_01X01, P23 CONN_01X01, P24 CONN_01X02, P25 CONN_01X03, P26 CONN_01X03, P27 CONN_01X02, P28 CONN_01X02, P29 CONN_01X02, P3 CONN_01X03, P30 CONN_01X02, P4 CONN_01X03, P5 CONN_02X07, P6 CONN_01X01, P7 CONN_01X01, P8 CONN_01X01, P9 CONN_01X01, U1 LTC2351-14, U10 MAX3463, U11 MAX3463, U12 MAX3463, U13 MAX3463, U14 MAX3463, U15 Si8261BCD-C-IS, U16 TS321, U17 Si8261BCD-C-IS, U18 Si8261BCD-C-IS, U19 AD8226, U2 XC6SLXN-TQG144, U20 AD8226, U21 AD8226, U22 LTC2351-14, U23 LT3010, U24 Si8261BCD-C-IS, U25 AMC1204, U26 OKR_T3, U27 Si8261BCD-C-IS, U28 ACS722KMATR-20AB-T, U29 MAX3463, U3 W25Q80DV, U30 MAX3463, U31 MAX3463, U32 MAX3463, U33 MAX3463, U34 Si8261BCD-C-IS, U35 Si8261BCD-C-IS, U36 ACS722KMATR-20AB-T, U37 TS321, U38 AD8226, U39 AD8226, U4 KSZ9031RNXCA, U40 AD8226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

Commit message: Backup
Parts:
- removed C121, C124, C125: 100nF, 00_Passives:C0603
- added C132: 100nF, 00_Passives:C0603, F.Cu at (83.8, 70.5)
- added C133: 100nF, 00_Passives:C0603, F.Cu at (55.0, 88.2)
- added C134: 100nF, 00_Passives:C0603, B.Cu at (75.5, 93.2)
- added C135: 100nF, 00_Passives:C0603, F.Cu at (84.2, 95.0)
- added C136: 100nF, 00_Passives:C0603, F.Cu at (159.5, 95.8)
- added C137: 100nF, 00_Passives:C0603, B.Cu at (61.8, 131.5)
- added C138: 100nF, 00_Passives:C0603, F.Cu at (106.8, 99.5)
- added C139: 100nF, 00_Passives:C0603, F.Cu at (76.2, 96.2)
- added C140: 100nF, 00_Passives:C0603, B.Cu at (58.0, 78.8)
- added C141: 100nF, 00_Passives:C0603, B.Cu at (73.8, 62.5)
- added C142: 100nF, 00_Passives:C0603, B.Cu at (52.5, 83.5)
- added C143: 100nF, 00_Passives:C0603, B.Cu at (71.2, 59.8)
- added C144: 100nF, 00_Passives:C0603, B.Cu at (55.0, 83.5)
- added C145: 100nF, 00_Passives:C0603, B.Cu at (58.0, 83.0)
- added C146: 100nF, 00_Passives:C0603, B.Cu at (72.8, 59.8)
- added C147: 100nF, 00_Passives:C0603, F.Cu at (51.0, 84.5)
- added C148: 100nF, 00_Passives:C0603, B.Cu at (58.0, 81.0)
- added C149: 100nF, 00_Passives:C0603, B.Cu at (71.8, 66.8)
- added C150: 100nF, 00_Passives:C0603, F.Cu at (66.8, 67.8)
- added C151: 100nF, 00_Passives:C0603, B.Cu at (57.0, 76.2)
- added C152: 100nF, 00_Passives:C0603, B.Cu at (70.8, 66.8)
- added C153: 100nF, 00_Passives:C0603, B.Cu at (73.8, 64.2)
- added C154: 100nF, 00_Passives:C0603, F.Cu at (108.5, 103.5)
- added C155: 100nF, 00_Passives:C0603, B.Cu at (67.2, 107.5)
- added C156: 100nF, 00_Passives:C0603, F.Cu at (69.2, 106.5)
- added C157: 10uF, 00_Passives:C1210, B.Cu at (87.8, 61.2)
- added C158: 10uF, 00_Passives:C1210, B.Cu at (87.8, 56.8)
- added C159: 100uF/16V, Capacitors_SMD:c_elec_6.3x5.3, F.Cu at (92.8, 59.0)
- added C160: 100nF, 00_Passives:C0603, B.Cu at (69.2, 66.8)
- added C161: 100nF, 00_Passives:C0603, B.Cu at (39.5, 65.2)
- added C163: 100nF, 00_Passives:C0603, B.Cu at (71.2, 72.2)
- added HOLE1: HOLE, 00_Local:hole_3mm, F.Cu at (234.8, 100.0)
- added HOLE10: HOLE, 00_Local:hole_3mm, F.Cu at (218.0, 53.0)
- added HOLE11: HOLE, 00_Local:hole_3mm, F.Cu at (138.0, 147.0)
- added HOLE2: HOLE, 00_Local:hole_3mm, F.Cu at (101.8, 122.0)
- added HOLE3: HOLE, 00_Local:hole_3mm, F.Cu at (194.8, 100.0)
- added HOLE4: HOLE, 00_Local:hole_3mm, F.Cu at (154.8, 100.0)
- added HOLE5: HOLE, 00_Local:hole_3mm, F.Cu at (101.8, 78.0)
- added HOLE6: HOLE, 00_Local:hole_3mm, F.Cu at (138.0, 53.0)
- added HOLE7: HOLE, 00_Local:hole_3mm, F.Cu at (218.0, 147.0)
- added HOLE8: HOLE, 00_Local:hole_3mm, F.Cu at (178.0, 53.0)
- added HOLE9: HOLE, 00_Local:hole_3mm, F.Cu at (178.0, 147.0)
- added R139: 1.0k, 00_Passives:R0603, F.Cu at (67.8, 96.8)
- added R140: 1.8k, 00_Passives:R0603, B.Cu at (83.8, 56.2)
- added R141: 150, 00_Passives:R0603, B.Cu at (83.8, 58.8)
- added U62: OKR_T3, 00_Passives:okr_t3, F.Cu at (85.2, 59.0)
- C100, C103, C107, C111, C94, C95, C98, C99, M13: moved to F.Cu
- C116, C17, L2, L3, L4: moved to B.Cu
- moved C116 146.2 mm to (67.2, 105.8)
- moved C120 122.8 mm to (51.2, 112.8)
- moved P26 78.8 mm to (77.8, 136.2), turned to 0 degrees
- moved C117 72.5 mm to (66.5, 102.5)
- moved D5 62.7 mm to (79.8, 129.8), turned to 270 degrees
- moved M13 59.4 mm to (77.8, 122.5), turned to 270 degrees
- moved P25 58.0 mm to (77.8, 125.7), turned to 0 degrees
- moved C98 35.1 mm to (65.8, 114.8), turned to 270 degrees
- moved U61 20.7 mm to (84.0, 68.0)
- moved R13 9.40 mm to (99.8, 87.2), turned to 0 degrees
- moved U57 6.59 mm to (163.1, 98.5)
- moved R11 6.19 mm to (99.8, 85.2), turned to 0 degrees
- moved P27 6.17 mm to (72.2, 125.5)
- moved P28 6.17 mm to (72.2, 131.2)
- moved P29 6.17 mm to (72.2, 136.8)
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Connections:
- C116 pad 1: GND -> +3.3V
- C116 pad 2: -5V -> GND
- C117 pad 1: GND -> +3.3V
- C117 pad 2: -5V -> GND
- C120 pad 1: GND -> +3.3V
- C120 pad 2: -5V -> GND
- P5 pad 1: +3.3V -> +2.5V
- U16 pad 2: -5V -> GND
- U2 pad 1: /FPGA/ETH_INT(1) -> /FPGA/SCL
- U2 pad 10: /FPGA/ETH_TX_CLK(1) -> /FPGA/ETH_RXD(1)(3)
- U2 pad 11: /FPGA/ETH_TXD(1)(3) -> /FPGA/ETH_TX_EN(1)
- U2 pad 112: /FPGA/HB_L0 -> /FPGA/HB_L2
- U2 pad 115: /FPGA/HB_L2 -> /Drive_1/H2
- U2 pad 119: /Drive_1/H2 -> /Drive_1/H1
- U2 pad 12: /FPGA/ETH_TXD(1)(2) -> /FPGA/ETH_TX_CLK(1)
- U2 pad 121: /Drive_1/H1 -> /FPGA/HB_L0
- U2 pad 14: /FPGA/ETH_RX_CLK(1) -> /FPGA/ETH_TXD(1)(3)
- U2 pad 15: /FPGA/ETH_TXD(1)(1) -> /FPGA/ETH_TXD(1)(2)
- U2 pad 16: /FPGA/ETH_TXD(1)(0) -> /FPGA/ETH_RX_CLK(1)
- U2 pad 17: Net-(U2-Pad17) -> /FPGA/ETH_TXD(1)(1)
- U2 pad 2: /FPGA/ETH_RX_DV(1) -> /FPGA/SDA
- U2 pad 21: Net-(U2-Pad21) -> /FPGA/ETH_TXD(1)(0)
- U2 pad 22: /FPGA/AUX_STR -> /FPGA/ETH_RESET(0)
- U2 pad 23: /FPGA/ETH_RESET(0) -> /FPGA/ETH_INT(0)
- U2 pad 33: /FPGA/SCL -> Net-(U2-Pad33)
- U2 pad 34: /FPGA/SDA -> Net-(U2-Pad34)
- U2 pad 5: /FPGA/ETH_RXD(1)(0) -> /FPGA/ETH_INT(1)
- U2 pad 6: /FPGA/ETH_RXD(1)(1) -> /FPGA/ETH_RX_DV(1)
- U2 pad 7: /FPGA/ETH_RXD(1)(2) -> /FPGA/ETH_RXD(1)(0)
- U2 pad 8: /FPGA/ETH_RXD(1)(3) -> /FPGA/ETH_RXD(1)(1)
- U2 pad 9: /FPGA/ETH_TX_EN(1) -> /FPGA/ETH_RXD(1)(2)
- U2 pad 92: /FPGA/FAN -> Net-(U2-Pad92)
- U2 pad 93: /FPGA/ETH_INT(0) -> /FPGA/AUX_STR
- U2 pad 97: /FPGA/HB_DISABLE -> /FPGA/FAN
- U37 pad 2: -5V -> GND
- U46 pad 2: -5V -> GND
- U47 pad 2: -5V -> GND
- U55 pad 2: -5V -> GND
- U56 pad 2: -5V -> GND
- U60 pad 1: Net-(U60-Pad1) -> GND
- U60 pad 4: Net-(U60-Pad1) -> GND
- U60 pad 8: Net-(U60-Pad1) -> GND
- U60 pad 9: Net-(U60-Pad1) -> GND
Routing:
- net +3.3V: track 301.9 -> 778.3 mm, vias 25 -> 37
- net +2.5V: track 38.0 -> 288.6 mm, vias 2 -> 13
- net +5V: track 142.0 -> 316.0 mm, vias 6 -> 9
- net /Drive_1/ISOL_15V: track 11.5 -> 163.8 mm
- net /Drive_2/ISOL_15V: track 11.8 -> 158.5 mm
- net +12V: track 78.8 -> 206.5 mm
- net -5V: track 127.2 -> 0.00 mm, vias 6 -> 0
- net GND: track 304.6 -> 430.1 mm, vias 58 -> 123
- net +1.2V: track 23.9 -> 139.6 mm, vias 5 -> 16
- net /Drive_2/BRIDGE-: track 56.8 -> 152.2 mm, vias 30 -> 41
- net +3.3VADC: track 11.4 -> 56.2 mm, vias 0 -> 2
- net /FPGA/FAN: track 0.00 -> 41.2 mm
- net /FPGA/MDC: track 0.00 -> 35.5 mm, vias 0 -> 3
- net /FPGA/MDIO: track 0.00 -> 32.9 mm, vias 0 -> 3
- net /Drive_1/BRIDGE-: track 79.3 -> 107.9 mm, vias 39 -> 46
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- added copper zone on B.Cu, net +1.2V
- added copper zone on F.Cu, net +3.3V
- added copper zone on B.Cu, net /Drive_1/BRIDGE-
- added copper zone on In2.Cu, net /Drive_1/BRIDGE-
- added copper zone on B.Cu, net /Drive_2/BRIDGE-
- added copper zone on In2.Cu, net /Drive_2/BRIDGE-
- added copper zone on B.Cu, net GND
- added copper zone on In2.Cu, net GND
Other:
- net class Default: clearance 0.125 -> 0.12
- net class iso added: clearance 7, trace_width 0.125, via_dia 0.6, via_drill 0.4
- rule trace_clearance: 0.125 -> 0.12

Commit message: First small drive hardware.
Parts:
- moved C70 34.8 mm to (92.8, 144.0)
- moved C72 7.00 mm to (87.5, 114.0)
- moved C75 7.00 mm to (87.5, 125.0)
- moved C76 7.00 mm to (87.5, 136.0)
- moved C79 7.00 mm to (87.5, 109.2)
- moved C80 7.00 mm to (87.5, 120.2)
- moved C81 7.00 mm to (87.5, 131.2)
- moved C84 7.00 mm to (92.8, 111.8)
- moved C85 7.00 mm to (92.8, 122.8)
- moved C86 7.00 mm to (92.8, 133.8)
- moved R105 7.00 mm to (83.8, 108.0)
- moved R106 7.00 mm to (83.8, 111.0)
- moved R107 7.00 mm to (83.5, 119.0)
- moved R108 7.00 mm to (83.5, 122.0)
- moved R109 7.00 mm to (83.5, 130.0)
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Routing:
- net +3.3V: track 778.3 -> 734.8 mm, vias 37 -> 34
- net +12V: track 206.5 -> 182.3 mm
- net Net-(P4-Pad2): track 48.8 -> 35.1 mm
- net +2.5V: track 288.6 -> 275.7 mm, vias 13 -> 11
- net GND: track 430.1 -> 441.9 mm, vias 123 -> 126
- net +1.2V: track 139.6 -> 127.9 mm, vias 16 -> 17
- net Net-(R133-Pad2): track 103.0 -> 109.9 mm
- net Net-(R134-Pad2): track 107.0 -> 113.6 mm
- net Net-(D2-Pad4): track 4.16 -> 9.84 mm
- net /FPGA/FAN: track 41.2 -> 45.5 mm, vias 0 -> 2
- net Net-(R124-Pad1): track 129.3 -> 125.1 mm
- net /FPGA/TRXB0_P: track 16.1 -> 20.4 mm
- net Net-(R132-Pad2): track 100.4 -> 104.6 mm
- net /Drive_1/ENC4_N: track 15.6 -> 11.9 mm
- net /Drive_1/ENC0_N: track 17.7 -> 13.9 mm
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- added copper zone on B.Cu, net +3.3V
