File: hardware/powerr.sch (KiCad schematic (older format))
At the start: 33 parts, among them CON1 BARREL_JACK, U26 OKR_T3, U41 OKR_T3, U45 OKR_T3, U50 LT3010, X3 RKZ1215D

Commit message: Progress.
Parts:
- removed CON1: BARREL_JACK, 00_Passives:smd_barrel_jack, symbol BARREL_JACK
- added P24: CONN_01X02, 00_Passives:FCI_02_5mm, symbol CONN_01X02
Connections:
- net +12V: now also P24.1 (P1)
- net GND: now also P24.2 (P2)
Changed lines of the file:
@@
 $EndDescr
-$Comp
-L BARREL_JACK CON1
-U 1 1 56D49D93
-P 1850 2750
-F 0 "CON1" H 1850 3000 60  0000 C CNN
-F 1 "BARREL_JACK" H 1850 2550 60  0000 C CNN
-F 2 "00_Passives:smd_barrel_jack" H 1850 2750 60  0001 C CNN
-F 3 "" H 1850 2750 60  0000 C CNN
-	1    1850 2750
-	1    0    0    -1
-$EndComp
 $Comp
 L OKR_T3 U41
@@
 	1    0    0    -1
 $EndComp
-$Comp
-L +3.3V #PWR48
-U 1 1 56D49EC2
-P 5150 3250
-F 0 "#PWR48" H 5150 3100 50  0001 C CNN
-F 1 "+3.3V" H 5150 3390 50  0000 C CNN
-F 2 "" H 5150 3250 50  0000 C CNN
-F 3 "" H 5150 3250 50  0000 C CNN
-	1    5150 3250
-	1    0    0    -1
-$EndComp
 Wire Wire Line
 	5150 3250 5150 3300
@@
 	5050 3300 5650 3300
 $Comp
-L GND #PWR34
+L GND #PWR44
 U 1 1 56D49EE6
 P 4400 5200
-F 0 "#PWR34" H 4400 4950 50  0001 C CNN
+F 0 "#PWR44" H 4400 4950 50  0001 C CNN
 F 1 "GND" H 4400 5050 50  0000 C CNN
 F 2 "" H 4400 5200 50  0000 C CNN
@@
 Connection ~ 4400 5150
 $Comp
-L +12V #PWR25
+L +12V #PWR31
 U 1 1 56D49FA0
 P 3600 3250
-F 0 "#PWR25" H 3600 3100 50  0001 C CNN
+F 0 "#PWR31" H 3600 3100 50  0001 C CNN
 F 1 "+12V" H 3600 3390 50  0000 C CNN
 F 2 "" H 3600 3250 50  0000 C CNN
@@
 	5050 5650 6250 5650
 $Comp
-L GND #PWR37
+L GND #PWR47
 U 1 1 56D4A185
 P 4400 7550
-F 0 "#PWR37" H 4400 7300 50  0001 C CNN
+F 0 "#PWR47" H 4400 7300 50  0001 C CNN
 F 1 "GND" H 4400 7400 50  0000 C CNN
 F 2 "" H 4400 7550 50  0000 C CNN
@@
 Connection ~ 4400 7500
 $Comp
-L +12V #PWR27
+L +12V #PWR33
 U 1 1 56D4A19E
 P 3600 5600
-F 0 "#PWR27" H 3600 5450 50  0001 C CNN
+F 0 "#PWR33" H 3600 5450 50  0001 C CNN
 F 1 "+12V" H 3600 5740 50  0000 C CNN
 F 2 "" H 3600 5600 50  0000 C CNN
@@
 	3600 5650 3750 5650
 $Comp
-L +5V #PWR49
+L +5V #PWR62
 U 1 1 56D4A1DA
 P 5150 5600
-F 0 "#PWR49" H 5150 5450 50  0001 C CNN
+F 0 "#PWR62" H 5150 5450 50  0001 C CNN
 F 1 "+5V" H 5150 5740 50  0000 C CNN
 F 2 "" H 5150 5600 50  0000 C CNN
@@
 $EndComp
 $Comp
-L GND #PWR31
+L GND #PWR41
 U 1 1 56D4A629
 P 4400 2850
-F 0 "#PWR31" H 4400 2600 50  0001 C CNN
+F 0 "#PWR41" H 4400 2600 50  0001 C CNN
 F 1 "GND" H 4400 2700 50  0000 C CNN
 F 2 "" H 4400 2850 50  0000 C CNN
@@
 Connection ~ 4400 2800
 $Comp
-L +12V #PWR23
+L +12V #PWR29
 U 1 1 56D4A642
 P 3600 900
-F 0 "#PWR23" H 3600 750 50  0001 C CNN
+F 0 "#PWR29" H 3600 750 50  0001 C CNN
 F 1 "+12V" H 3600 1040 50  0000 C CNN
 F 2 "" H 3600 900 50  0000 C CNN
@@
 	3600 950  3750 950
 $Comp
-L +1.2V #PWR47
+L +1.2V #PWR60
 U 1 1 56D4A685
 P 5150 900
-F 0 "#PWR47" H 5150 1040 20  0001 C CNN
+F 0 "#PWR60" H 5150 1040 20  0001 C CNN
 F 1 "+1.2V" H 5150 1010 30  0000 C CNN
 F 2 "" H 5150 900 60  0000 C CNN
@@
 $EndComp
 $Comp
-L +3.3VADC #PWR82
+L +3.3VADC #PWR99
 U 1 1 56D4B08E
 P 7700 5600
-F 0 "#PWR82" H 7850 5550 50  0001 C CNN
+F 0 "#PWR99" H 7850 5550 50  0001 C CNN
 F 1 "+3.3VADC" H 7700 5700 50  0000 C CNN
 F 2 "" H 7700 5600 50  0000 C CNN
@@
 Connection ~ 6200 5650
 $Comp
-L GND #PWR74
+L GND #PWR91
 U 1 1 56D4B154
 P 6900 6600
-F 0 "#PWR74" H 6900 6350 50  0001 C CNN
+F 0 "#PWR91" H 6900 6350 50  0001 C CNN
 F 1 "GND" H 6900 6450 50  0000 C CNN
 F 2 "" H 6900 6600 50  0000 C CNN
@@
 Connection ~ 7700 6250
 $Comp
-L GND #PWR83
+L GND #PWR100
 U 1 1 56D4BB5E
 P 7700 6850
-F 0 "#PWR83" H 7700 6600 50  0001 C CNN
+F 0 "#PWR100" H 7700 6600 50  0001 C CNN
 F 1 "GND" H 7700 6700 50  0000 C CNN
 F 2 "" H 7700 6850 50  0000 C CNN
@@
 	7700 6850 7700 6800
 $Comp
-L +12V #PWR10
+L +12V #PWR11
 U 1 1 56D4C0A6
 P 2300 2600
-F 0 "#PWR10" H 2300 2450 50  0001 C CNN
+F 0 "#PWR11" H 2300 2450 50  0001 C CNN
 F 1 "+12V" H 2300 2740 50  0000 C CNN
 F 2 "" H 2300 2600 50  0000 C CNN
@@
 	2150 2650 2950 2650
 $Comp
-L GND #PWR11
+L GND #PWR12
 U 1 1 56D4C114
 P 2300 2950
-F 0 "#PWR11" H 2300 2700 50  0001 C CNN
+F 0 "#PWR12" H 2300 2700 50  0001 C CNN
 F 1 "GND" H 2300 2800 50  0000 C CNN
 F 2 "" H 2300 2950 50  0000 C CNN
@@
 	1    0    0    -1
 $EndComp
-Wire Wire Line
-	2150 2750 2300 2750
-Wire Wire Line
-	2300 2750 2300 2950
-Wire Wire Line
-	2150 2850 2300 2850
-Connection ~ 2300 2850
 $Comp
 L C C81
@@
 Connection ~ 5250 3300
 $Comp
-L GND #PWR51
+L GND #PWR64
 U 1 1 56D4C7DD
 P 5250 3850
-F 0 "#PWR51" H 5250 3600 50  0001 C CNN
+F 0 "#PWR64" H 5250 3600 50  0001 C CNN
 F 1 "GND" H 5250 3700 50  0000 C CNN
 F 2 "" H 5250 3850 50  0000 C CNN
@@
 	5250 3800 5250 3850
 $Comp
-L GND #PWR56
+L GND #PWR68
 U 1 1 56D4C7FB
 P 5650 3850
-F 0 "#PWR56" H 5650 3600 50  0001 C CNN
+F 0 "#PWR68" H 5650 3600 50  0001 C CNN
 F 1 "GND" H 5650 3700 50  0000 C CNN
 F 2 "" H 5650 3850 50  0000 C CNN
@@
 	5650 3800 5650 3850
 $Comp
-L GND #PWR85
+L GND #PWR103
 U 1 1 56D4C8C1
 P 8200 6150
-F 0 "#PWR85" H 8200 5900 50  0001 C CNN
+F 0 "#PWR103" H 8200 5900 50  0001 C CNN
 F 1 "GND" H 8200 6000 50  0000 C CNN
 F 2 "" H 8200 6150 50  0000 C CNN
@@
 	8200 6100 8200 6150
 $Comp
-L GND #PWR87
+L GND #PWR104
 U 1 1 56D4C8C8
 P 8600 6150
-F 0 "#PWR87" H 8600 5900 50  0001 C CNN
+F 0 "#PWR104" H 8600 5900 50  0001 C CNN
 F 1 "GND" H 8600 6000 50  0000 C CNN
 F 2 "" H 8600 6150 50  0000 C CNN
@@
 Connection ~ 8200 5650
 $Comp
-L GND #PWR52
+L GND #PWR65
 U 1 1 56D4C9FA
 P 5250 6250
-F 0 "#PWR52" H 5250 6000 50  0001 C CNN
+F 0 "#PWR65" H 5250 6000 50  0001 C CNN
 F 1 "GND" H 5250 6100 50  0000 C CNN
 F 2 "" H 5250 6250 50  0000 C CNN
@@
 	5250 6200 5250 6250
 $Comp
-L GND #PWR59
+L GND #PWR72
 U 1 1 56D4CA01
 P 5950 6250
-F 0 "#PWR59" H 5950 6000 50  0001 C CNN
+F 0 "#PWR72" H 5950 6000 50  0001 C CNN
 F 1 "GND" H 5950 6100 50  0000 C CNN
 F 2 "" H 5950 6250 50  0000 C CNN
@@
 Connection ~ 5250 950
 $Comp
-L GND #PWR50
+L GND #PWR63
 U 1 1 56D4D30E
 P 5250 1500
-F 0 "#PWR50" H 5250 1250 50  0001 C CNN
+F 0 "#PWR63" H 5250 1250 50  0001 C CNN
 F 1 "GND" H 5250 1350 50  0000 C CNN
 F 2 "" H 5250 1500 50  0000 C CNN
@@
 	5250 1450 5250 1500
 $Comp
-L GND #PWR55
+L GND #PWR67
 U 1 1 56D4D315
 P 5650 1500
-F 0 "#PWR55" H 5650 1250 50  0001 C CNN
+F 0 "#PWR67" H 5650 1250 50  0001 C CNN
 F 1 "GND" H 5650 1350 50  0000 C CNN
 F 2 "" H 5650 1500 50  0000 C CNN
@@
 $EndComp
 $Comp
-L GND #PWR12
+L GND #PWR13
 U 1 1 56D4D996
 P 2550 3150
-F 0 "#PWR12" H 2550 2900 50  0001 C CNN
+F 0 "#PWR13" H 2550 2900 50  0001 C CNN
 F 1 "GND" H 2550 3000 50  0000 C CNN
 F 2 "" H 2550 3150 50  0000 C CNN
@@
 	2550 3100 2550 3150
 $Comp
-L GND #PWR13
+L GND #PWR15
 U 1 1 56D4D99D
 P 2950 3150
-F 0 "#PWR13" H 2950 2900 50  0001 C CNN
+F 0 "#PWR15" H 2950 2900 50  0001 C CNN
 F 1 "GND" H 2950 3000 50  0000 C CNN
 F 2 "" H 2950 3150 50  0000 C CNN
@@
 $EndComp
 $Comp
-L GND #PWR24
+L GND #PWR30
 U 1 1 56D4DB48
 P 3600 1800
-F 0 "#PWR24" H 3600 1550 50  0001 C CNN
+F 0 "#PWR30" H 3600 1550 50  0001 C CNN
 F 1 "GND" H 3600 1650 50  0000 C CNN
 F 2 "" H 3600 1800 50  0000 C CNN
@@
 $EndComp
 $Comp
-L GND #PWR26
+L GND #PWR32
 U 1 1 56D4DBBB
 P 3600 4100
-F 0 "#PWR26" H 3600 3850 50  0001 C CNN
+F 0 "#PWR32" H 3600 3850 50  0001 C CNN
 F 1 "GND" H 3600 3950 50  0000 C CNN
 F 2 "" H 3600 4100 50  0000 C CNN
@@
 $EndComp
 $Comp
-L GND #PWR28
+L GND #PWR34
 U 1 1 56D4DC2D
 P 3600 6450
-F 0 "#PWR28" H 3600 6200 50  0001 C CNN
+F 0 "#PWR34" H 3600 6200 50  0001 C CNN
 F 1 "GND" H 3600 6300 50  0000 C CNN
 F 2 "" H 3600 6450 50  0000 C CNN
@@
 $EndComp
 $Comp
-L +15V #PWR41
+L +15V #PWR54
 U 1 1 56D4EC18
 P 4900 7800
-F 0 "#PWR41" H 4900 7760 30  0001 C CNN
+F 0 "#PWR54" H 4900 7760 30  0001 C CNN
 F 1 "+15V" H 4900 7910 30  0000 C CNN
 F 2 "" H 4900 7800 60  0000 C CNN
@@
 $EndComp
 $Comp
-L -15V #PWR42
+L -15V #PWR55
 U 1 1 56D4EC7D
 P 4900 8900
-F 0 "#PWR42" H 4900 9030 20  0001 C CNN
+F 0 "#PWR55" H 4900 9030 20  0001 C CNN
 F 1 "-15V" H 4900 9000 30  0000 C CNN
 F 2 "" H 4900 8900 60  0000 C CNN
@@
 	4900 7800 4900 8250
 $Comp
-L GND #PWR57
+L GND #PWR69
 U 1 1 56D4EE79
 P 5700 8350
-F 0 "#PWR57" H 5700 8100 50  0001 C CNN
+F 0 "#PWR69" H 5700 8100 50  0001 C CNN
 F 1 "GND" H 5700 8200 50  0000 C CNN
 F 2 "" H 5700 8350 50  0000 C CNN
@@
 	4750 8350 5700 8350
 $Comp
-L +12V #PWR15
+L +12V #PWR19
 U 1 1 56D4F097
 P 3450 8200
-F 0 "#PWR15" H 3450 8050 50  0001 C CNN
+F 0 "#PWR19" H 3450 8050 50  0001 C CNN
 F 1 "+12V" H 3450 8340 50  0000 C CNN
 F 2 "" H 3450 8200 50  0000 C CNN
@@
 $EndComp
 $Comp
-L GND #PWR16
+L GND #PWR20
 U 1 1 56D4F0A5
 P 3450 8800
-F 0 "#PWR16" H 3450 8550 50  0001 C CNN
+F 0 "#PWR20" H 3450 8550 50  0001 C CNN
 F 1 "GND" H 3450 8650 50  0000 C CNN
 F 2 "" H 3450 8800 50  0000 C CNN
@@
 $EndComp
 $Comp
-L GND #PWR54
+L GND #PWR66
 U 1 1 56D563CB
 P 5550 6250
-F 0 "#PWR54" H 5550 6000 50  0001 C CNN
+F 0 "#PWR66" H 5550 6000 50  0001 C CNN
 F 1 "GND" H 5550 6100 50  0000 C CNN
 F 2 "" H 5550 6250 50  0000 C CNN
@@
 	5550 5800 5550 5650
 Connection ~ 5550 5650
+$Comp
+L +3.3V #PWR61
+U 1 1 56DC09FA
+P 5150 3250
+F 0 "#PWR61" H 5200 3280 20  0001 C CNN
+F 1 "+3.3V" H 5150 3340 30  0000 C CNN
+F 2 "" H 5150 3250 60  0000 C CNN
+F 3 "" H 5150 3250 60  0000 C CNN
+	1    5150 3250
+	1    0    0    -1
+$EndComp
+$Comp
+L CONN_01X02 P24
+U 1 1 56DC4E95
+P 1950 2700
+F 0 "P24" H 1950 2850 50  0000 C CNN
+F 1 "CONN_01X02" V 2050 2700 50  0000 C CNN
+F 2 "00_Passives:FCI_02_5mm" H 1950 2700 50  0001 C CNN
+F 3 "" H 1950 2700 50  0000 C CNN
+F 4 "1860166" H 1950 2700 60  0001 C CNN "Farnell"
+F 5 "FCI" H 1950 2700 60  0001 C CNN "Manufacturer"
+F 6 "20020109-G021A01LF" H 1950 2700 60  0001 C CNN "PartNr"
+F 7 "1859979" H 1950 2700 60  0001 C CNN "Farnell_mating"
+	1    1950 2700
+	-1   0    0    -1
+$EndComp
+Wire Wire Line
+	2150 2750 2300 2750
+Wire Wire Line
+	2300 2750 2300 2950
 $EndSCHEMATC

Commit message: Backup
Parts:
- added C116, C117, C120, C155, C156, C160, C161, C163: 100nF, 00_Passives:C0603, symbol C
- added C157, C158: 10uF, 00_Passives:C1210, symbol C
- added C159: 100uF/16V, Capacitors_SMD:c_elec_6.3x5.3, symbol CAPAPOL
- added HOLE1, HOLE2, HOLE3, HOLE4, HOLE5, HOLE? (x6): HOLE, 00_Local:hole_3mm, symbol HOLE
- added R140: 1.8k, 00_Passives:R0603, symbol R
- added R141: 150, 00_Passives:R0603, symbol R
- added U62: OKR_T3, 00_Passives:okr_t3, symbol OKR_T3
Connections:
- net labels added: +2.5V, ISO0, ISO1, ISO2, ISO3, ISO4, ISO5
- wire segments 93 -> 147
Other:
- note added: "Holes to connect heatsink to the middle ground plane"
- note added: "Isolated heatsink holes"

Commit message: First small drive hardware.
Parts:
- gave numbers to parts that had none: 6
Changed lines of the file:
@@
 Connection ~ 9900 8600
 $Comp
-L HOLE HOLE?
+L HOLE HOLE6
 U 1 1 56F34D98
 P 11600 7600
-F 0 "HOLE?" H 11600 7600 60  0000 C CNN
+F 0 "HOLE6" H 11600 7600 60  0000 C CNN
 F 1 "HOLE" H 11600 7600 60  0000 C CNN
 F 2 "00_Local:hole_3mm" H 11600 7600 60  0001 C CNN
@@
 Isolated heatsink holes
 $Comp
-L HOLE HOLE?
+L HOLE HOLE8
 U 1 1 56F350D1
 P 11950 7600
-F 0 "HOLE?" H 11950 7600 60  0000 C CNN
+F 0 "HOLE8" H 11950 7600 60  0000 C CNN
 F 1 "HOLE" H 11950 7600 60  0000 C CNN
 F 2 "00_Local:hole_3mm" H 11950 7600 60  0001 C CNN
@@
 	11950 7800 11950 8100
 $Comp
-L HOLE HOLE?
+L HOLE HOLE10
 U 1 1 56F3511E
 P 12300 7600
-F 0 "HOLE?" H 12300 7600 60  0000 C CNN
+F 0 "HOLE10" H 12300 7600 60  0000 C CNN
 F 1 "HOLE" H 12300 7600 60  0000 C CNN
 F 2 "00_Local:hole_3mm" H 12300 7600 60  0001 C CNN
@@
 	12300 7800 12300 8100
 $Comp
-L HOLE HOLE?
+L HOLE HOLE7
 U 1 1 56F351DA
 P 11600 8350
-F 0 "HOLE?" H 11600 8350 60  0000 C CNN
+F 0 "HOLE7" H 11600 8350 60  0000 C CNN
 F 1 "HOLE" H 11600 8350 60  0000 C CNN
 F 2 "00_Local:hole_3mm" H 11600 8350 60  0001 C CNN
@@
 	11600 8550 11600 8850
 $Comp
-L HOLE HOLE?
+L HOLE HOLE9
 U 1 1 56F351E1
 P 11950 8350
-F 0 "HOLE?" H 11950 8350 60  0000 C CNN
+F 0 "HOLE9" H 11950 8350 60  0000 C CNN
 F 1 "HOLE" H 11950 8350 60  0000 C CNN
 F 2 "00_Local:hole_3mm" H 11950 8350 60  0001 C CNN
@@
 	11950 8550 11950 8850
 $Comp
-L HOLE HOLE?
+L HOLE HOLE11
 U 1 1 56F351E8
 P 12300 8350
-F 0 "HOLE?" H 12300 8350 60  0000 C CNN
+F 0 "HOLE11" H 12300 8350 60  0000 C CNN
 F 1 "HOLE" H 12300 8350 60  0000 C CNN
 F 2 "00_Local:hole_3mm" H 12300 8350 60  0001 C CNN
