File: small_drive/small_drive.sch (KiCad schematic (older format))
At the start: 155 parts, among them J1 DB9, J2 DB15, M1 SiR826DP, M2 SiR826DP, M3 SiR826DP, M4 SiR826DP, M5 SiR826DP, M6 SiR826DP, P1 CONN_01X04, P2 CONN_01X04, P3 CONN_01X04, P5 CONN_01X02, P6 CONN_01X02, P7 CONN_01X02, U1 XMC4400-F64x512, U10 LM5106, U11 ACS711KLCTR-12AB-T, U12 ACS711ELCTR-25AB-T, U13 ACS711KLCTR-12AB-T, U14 AD8226, U15 MAX3096, U16 AMC1203, U17 7805, U18 LT1764EQ, U19 KSZ8081, U2 ips511g, U20 ETH100_MAG, U3 ips511g, U4 LTC2850, U5 AD8226, U6 LT1764EQ, U7 MC33074DTBR2, U8 LM5106, U9 LM5106, X1 NKE1212DC, X2 NKE1212DC, X3 HCPL0201, X4 HCPL0201, X5 HCPL0201, X6 HCPL0201, Y1 12MHz, Y2 25MHz

Commit message: Pauze backup
Parts:
- added P4: CONN_01X04, Pin_Headers:Pin_Header_Straight_1x04, symbol CONN_01X04
- added P8: CONN_01X01, Pin_Headers:Pin_Header_Straight_1x01, symbol CONN_01X01
- added R47, R48: 10k, Resistors_SMD:R_0603, symbol R
- P1: footprint Connect:bornier4 -> 00_Passives:PC_drive_5.25_conn
Connections:
- wire segments 650 -> 900
Other:
- note added: "FIXME:\n\n1. Debugging pins\n2. reset circuit\n3. pinning xmc4500 checken.\n"
- note added: "P0.1 ETH0 CRS_DVB\nP0.0 U1C1 DX0D\nP14.14 VADC G1CH6\nP14.7 VADC G0CH7 POSIF0 IN0B\nP14.6 VADC G0CH6 POSIF0 IN1B"
- note added: "P0.3 HRPWM0_OUT01/CCU80_OUT01\nP0.5 HRPWM0_OUT00/CCU80_OUT00\nP0.6 HRPWM0_OUT30 (sync?)\nP1.8 DSD_MCLK 1A 0D 2D 3D\nP1.1 POSIF0_IN2A (ENC_Z)\nP1.2 POSIF0_IN1A (ENC_B)\nP1.3 POSIF0_IN0A (ENC_A)"
- note added: "P14.4 VADC G2CH0\nP14.0 VADC G0CH0\nP14.8 VADC G1CH0\nP2.9 ETH0 TXD1\nP2.8 ETH0 TXD0\nP2.5 ETH0 TX_EN\nP2.4 ETH0 RXERA\nP2.3 ETH0 RXD1A\nP2.2 ETH0 RXD0A"
- note added: "P2.1 ETH0_CLKRMIIA\nP2.0 ETH0_MDO MDIB\nP2.7 ETH0_MDC\nP2.6 DSD_IN1B\nP1.5 U0C0_DOUT0\nP1.4 U0C0_DX0B"
- note removed: "FIXME:\n\n1. Debugging pins\n2. 1.65V ref voor sincos.\n3. pinning xmc4500 checken."
- moved on the sheet: C2, C35, C4, C44, C45, C46, C47, C5, C50, C51, D1A, D1B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

Commit message: PCB ordered.
Connections:
- net labels added: SWCLK, SWDIO
Changed lines of the file:
@@
 Text Label 11850 4250 0    60   ~ 0
 LED3
-Text Label 2100 11750 0    60   ~ 0
+Text Label 2100 11350 0    60   ~ 0
 LED0
-Text Label 2100 10750 0    60   ~ 0
+Text Label 2100 11450 0    60   ~ 0
 LED1
-Text Label 2000 4500 0    60   ~ 0
+Text Label 2100 11750 0    60   ~ 0
 LED2
-Text Label 2000 4600 0    60   ~ 0
+Text Label 2100 11950 0    60   ~ 0
 LED3
 $Comp
@@
 	0    1    1    0
 $EndComp
-Text Label 2050 4300 0    60   ~ 0
+Text Label 2000 4300 0    60   ~ 0
 ETH_CRS_DVA
 Text Label 2050 8600 0    60   ~ 0
@@
 Text Label 8750 10250 0    60   ~ 0
 ENC_12V
-Text Label 2100 11450 0    60   ~ 0
+Text Label 2100 11250 0    60   ~ 0
 ENC_5V
 Text Label 2100 10850 0    60   ~ 0
@@
 Text Label 5750 6150 0    60   ~ 0
 ETH0_~RST
-Text Label 2100 11350 0    60   ~ 0
+Text Label 2100 10750 0    60   ~ 0
 ETH0_~RST
 $Comp
@@
 Text Label 10000 8450 1    60   ~ 0
 LED4
-Text Label 2100 11950 0    60   ~ 0
+Text Label 2000 4600 0    60   ~ 0
 LED4
 $Comp
@@
 Wire Wire Line
 	11900 5700 12850 5700
-Text Label 2100 11250 0    60   ~ 0
+Text Label 2000 4500 0    60   ~ 0
 HBEN
 Wire Wire Line
@@
 Wire Wire Line
 	12600 2850 12600 3100
-Text Notes 3000 11500 0    60   ~ 0
+Text Notes 3350 11500 0    60   ~ 0
 P0.3 HRPWM0_OUT01/CCU80_OUT01\nP0.5 HRPWM0_OUT00/CCU80_OUT00\nP0.6 HRPWM0_OUT30 (sync?)\nP1.8 DSD_MCLK 1A 0D 2D 3D\nP1.1 POSIF0_IN2A (ENC_Z)\nP1.2 POSIF0_IN1A (ENC_B)\nP1.3 POSIF0_IN0A (ENC_A)
 Text Notes 4800 9700 0    60   ~ 0
@@
 Wire Wire Line
 	17650 2950 18050 2950
+Text Label 2600 9500 0    60   ~ 0
+SWDIO
+Text Label 2600 9600 0    60   ~ 0
+SWCLK
 $EndSCHEMATC
