File: control_stage/control_stage.sch (KiCad schematic (older format))
At the start: 121 parts, among them J1 DB9, J2 DB15, P1 CONN_01X04, P2 CONN_01X04, P3 CONN_01X04, P4 CONN_01X04, P8 CONN_01X01, U1 XMC4400-F100, U14 AD8226, U15 MAX3463, U17 7805, U18 LT1764EQ, U19 KSZ8081, U2 ips511g, U20 ETH100_MAG, U21 MAX3463, U22 MAX3463, U23 MAX3463, U3 ips511g, U4 MAX3463, U5 AD8226, U6 LT1764EQ, U7 MC33074DTBR2, X1 NKE1212DC, X2 NKE1212DC, Y1 12MHz, Y2 25MHz

Commit message: Starting the control_stage (copied from small_drive)
Parts:
- removed C34, C36: 100uF/35V, Capacitors_SMD:c_elec_8x10.5, symbol small_drive-rescue:CP-RESCUE-small_drive
- removed C37, C52, C53, C54, C55: 100nF, Capacitors_SMD:C_0603, symbol small_drive-rescue:C-RESCUE-small_drive
- removed R6, R7, R8: 10k, Resistors_SMD:R_0603, symbol small_drive-rescue:R-RESCUE-small_drive
- removed U17: 7805, 00_Local:TO220_78xx, symbol small_drive-rescue:7805
- removed unit 1 of U7
- removed X2: NKE1212DC, 00_Local:NKE-SC, symbol small_drive-rescue:NKE1212DC
- C1, C14, C32, C38, C6: symbol small_drive-rescue:CP-RESCUE-small_drive -> CP-RESCUE-small_drive
- C10, C11, C12, C13, C15, C16, C17, C18, C28, C29, C3, C30, C31, C33, C39, C40, C41, C42, C43, C44, C45, C46, C47, C48, C49, C50, C51, C56, C57, C58, C59, C60, C61, C62, C7, C8, C9: symbol small_drive-rescue:C-RESCUE-small_drive -> C-RESCUE-small_drive
- D1: symbol small_drive-rescue:LED_592 -> LED_592
- HOLE1, HOLE2, HOLE3, HOLE4: symbol small_drive-rescue:HOLE -> HOLE
- J1: symbol small_drive-rescue:DB9 -> DB9
- J2: symbol small_drive-rescue:DB15 -> DB15
- P1, P2, P3, P4: symbol small_drive-rescue:CONN_01X04 -> CONN_01X04
- P8: symbol small_drive-rescue:CONN_01X01 -> CONN_01X01
- R1, R18, R19, R2, R20, R21, R22, R23, R24, R3, R35, R36, R37, R38, R39, R4, R40, R41, R42, R43, R44, R45, R46, R47, R48, R49, R5, R50, R51, R52, R53, R54, R55, R56, R57, R58, R59: symbol small_drive-rescue:R-RESCUE-small_drive -> R-RESCUE-small_drive
- U1: symbol small_drive-rescue:XMC4400-F100-RESCUE-small_drive -> XMC4400-F100-RESCUE-small_drive
- U14, U5: symbol small_drive-rescue:AD8226 -> AD8226
- U15, U21, U22, U23, U4: symbol small_drive-rescue:LTC2850-RESCUE-small_drive -> LTC2850-RESCUE-small_drive
- U18, U6: symbol small_drive-rescue:LT1764EQ -> LT1764EQ
- U19: symbol small_drive-rescue:KSZ8081 -> KSZ8081
- U2, U3: symbol small_drive-rescue:ips511g -> ips511g
- U20: symbol small_drive-rescue:ETH100_MAG -> ETH100_MAG
- U7: symbol small_drive-rescue:TL074-RESCUE-small_drive -> TL074-RESCUE-small_drive
- X1: symbol small_drive-rescue:NKE1212DC -> NKE1212DC
- Y1, Y2: symbol small_drive-rescue:Crystal -> Crystal
Connections:
- net labels removed: +12P, +5P, GNDPWR
- wire segments 694 -> 637

Commit message: Control stage, initial version.
Parts:
- C1, C14, C32, C38, C6: symbol CP-RESCUE-small_drive -> small_drive-rescue:CP-RESCUE-small_drive
- C10, C11, C12, C13, C15, C16, C17, C18, C28, C29, C3, C30, C31, C33, C39, C40, C41, C42, C43, C44, C45, C46, C47, C48, C49, C50, C51, C56, C57, C58, C59, C60, C61, C62, C7, C8, C9: symbol C-RESCUE-small_drive -> small_drive-rescue:C-RESCUE-small_drive
- D1: symbol LED_592 -> Local:LED_592
- HOLE1, HOLE2, HOLE3, HOLE4: symbol HOLE -> small_drive-rescue:HOLE
- J1: symbol DB9 -> small_drive-rescue:DB9
- J2: symbol DB15 -> small_drive-rescue:DB15
- P1, P2, P3, P4: symbol CONN_01X04 -> small_drive-rescue:CONN_01X04
- P8: symbol CONN_01X01 -> small_drive-rescue:CONN_01X01
- R1, R18, R19, R2, R20, R21, R22, R23, R24, R3, R35, R36, R37, R38, R39, R4, R40, R41, R42, R43, R44, R45, R46, R47, R48, R49, R5, R50, R51, R52, R53, R54, R55, R56, R57, R58, R59: symbol R-RESCUE-small_drive -> small_drive-rescue:R-RESCUE-small_drive
- U1: symbol XMC4400-F100-RESCUE-small_drive -> small_drive-rescue:XMC4400-F100-RESCUE-small_drive
- U14, U5: symbol AD8226 -> Local:AD8226
- U15, U21, U22, U23, U4: symbol LTC2850-RESCUE-small_drive -> small_drive-rescue:LTC2850-RESCUE-small_drive
- U18, U6: symbol LT1764EQ -> small_drive-rescue:LT1764EQ
- U19: symbol KSZ8081 -> Local:KSZ8081
- U2, U3: symbol ips511g -> Local:ips511g
- U20: symbol ETH100_MAG -> Local:ETH100_MAG
- U7: symbol TL074-RESCUE-small_drive -> small_drive-rescue:TL074-RESCUE-small_drive
- X1: symbol NKE1212DC -> Local:NKE1212DC
- Y1, Y2: symbol Crystal -> small_drive-rescue:Crystal
Connections:
- wire segments 637 -> 641
