File: hv_power/hv_power.kicad_pcb (KiCad board)
At the start: 2 copper layers, 100 x 100 mm, 114 parts, among them J1 Conn_01x01_Male, J10 Conn_02x03_Odd_Even, J11 Conn_02x03_Odd_Even, J12 Conn_02x03_Odd_Even, J13 Conn_02x04_Odd_Even, J14 Conn_01x01_Male, J2 Conn_01x01_Male, J3 Conn_01x01_Male, J4 V-, J5 V-, J6 V-, J7 V+, J8 V+, J9 V+, M1 NMOS_KELVIN, M2 NMOS_KELVIN, M3 NMOS_KELVIN, M4 NMOS_KELVIN, M5 NMOS_KELVIN, M6 NMOS_KELVIN, U1 UCC23511DWY, U17 THS4531, U2 UCC23511DWY, U26 THS4531, U29 THS4531, U3 UCC23511DWY, U4 UCC23511DWY, U5 UCC23511DWY, U6 UCC23511DWY

Commit message: Motor runs, encoder checksum does not work.
Other:
- net class Default removed

Commit message: Ordered new boards.
Parts:
- removed C21, C25, C26, C63, C67, C68, C73, C77, C78: 1uF, Capacitor_SMD:C_0805_2012Metric
- removed C27, C69, C79: 100nF, Capacitor_SMD:C_0603_1608Metric
- removed D2, D4, D6: STTH112A, 00_Passives:D_SMA
- removed J14: Conn_01x01_Male, TestPoint:TestPoint_Pad_1.0x1.0mm
- removed R17, R26, R62, R64, R75, R77: 4.7, Resistor_SMD:R_0603_1608Metric
- removed R60, R61, R73, R74, R86, R87: 51, Resistor_SMD:R_0603_1608Metric
- removed U17, U26, U29: THS4531, Package_SO:MSOP-8_3x3mm_P0.65mm
- added C3: C, Capacitor_SMD:C_1206_3216Metric, F.Cu at (177.3, 36.8)
- added C4: C, Capacitor_SMD:C_1206_3216Metric, F.Cu at (177.3, 66.8)
- added C5: C, Capacitor_SMD:C_1206_3216Metric, F.Cu at (177.3, 96.8)
- added R10: R, Resistor_SMD:R_1206_3216Metric, F.Cu at (172.7, 66.8)
- added R11: 270, Resistor_SMD:R_2512_6332Metric, F.Cu at (215.4, 66.5)
- added R12: R, Resistor_SMD:R_1206_3216Metric, F.Cu at (172.7, 96.8)
- added R13: 270, Resistor_SMD:R_2512_6332Metric, F.Cu at (215.5, 96.5)
- added R8: R, Resistor_SMD:R_1206_3216Metric, F.Cu at (172.7, 36.8)
- added R9: 270, Resistor_SMD:R_2512_6332Metric, F.Cu at (215.5, 36.5)
- added U7: TSV991ILT, Package_TO_SOT_SMD:SOT-23-5, F.Cu at (163.6, 54.3)
- added U8: TSV991ILT, Package_TO_SOT_SMD:SOT-23-5, F.Cu at (163.6, 84.3)
- added U9: TSV991ILT, Package_TO_SOT_SMD:SOT-23-5, F.Cu at (163.6, 114.3)
- C23, C32, C65, C70, C75, C80: footprint Capacitor_SMD:C_1206_3216Metric -> Capacitor_SMD:C_0805_2012Metric
- C92, C93, C94: footprint Capacitor_SMD:C_1812_4532Metric -> Capacitor_SMD:C_2220_5650Metric
- M1, M2, M3, M4, M5, M6: value NMOS_KELVIN -> TBD
- R27, R65, R78: footprint Resistor_SMD:R_0805_2012Metric -> Resistor_SMD:R_0603_1608Metric
- R31, R69, R82: footprint Resistor_SMD:R_0603_1608Metric -> Resistor_SMD:R_0805_2012Metric
- moved R27 8.00 mm to (162.5, 43.6), turned to 90 degrees
- moved R65 8.00 mm to (162.5, 73.6), turned to 90 degrees
- moved R78 8.00 mm to (162.5, 103.6), turned to 90 degrees
- moved R25 2.98 mm to (161.0, 43.6), turned to -90 degrees
- moved R63 2.98 mm to (161.0, 73.6), turned to -90 degrees
- moved R76 2.98 mm to (161.0, 103.6), turned to -90 degrees
- moved R34 2.50 mm to (160.6, 54.3)
- moved R72 2.50 mm to (160.6, 84.3)
- moved R85 2.50 mm to (160.6, 114.3)
- moved C66 2.43 mm to (159.1, 75.6), turned to 90 degrees
- moved C76 2.43 mm to (159.1, 105.6), turned to 90 degrees
- moved C24 2.43 mm to (159.1, 45.6), turned to 90 degrees
- moved D5 2.33 mm to (163.5, 67.3)
- moved D7 2.33 mm to (163.5, 97.3)
- moved D3 2.33 mm to (163.5, 37.3)
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Connections:
- net Net-(C1-Pad1) renamed /pe
- net Net-(J1-Pad1) renamed /H_Bridge0/sw_m2
- net Net-(J13-Pad8) renamed /ntc
- net Net-(J2-Pad1) renamed /H_Bridge1/sw_m2
- net Net-(J3-Pad1) renamed /H_Bridge2/sw_m2
- net Net-(JP1-Pad2) renamed /H_Bridge0/sw_m1
- net Net-(JP2-Pad2) renamed /H_Bridge1/sw_m1
- net Net-(JP3-Pad2) renamed /H_Bridge2/sw_m1
- net Net-(M1-PadG) renamed /H_Bridge0/sw_g
- net Net-(M3-PadG) renamed /H_Bridge1/sw_g
- net Net-(M5-PadG) renamed /H_Bridge2/sw_g
- net Net-(R2-Pad1) renamed /H_Bridge0/d1
- net Net-(R29-Pad2) renamed /H_Bridge0/sw_o
- net Net-(R3-Pad1) renamed /H_Bridge0/d2
- net Net-(R4-Pad1) renamed /H_Bridge1/d1
- net Net-(R5-Pad1) renamed /H_Bridge1/d2
- net Net-(R6-Pad1) renamed /H_Bridge2/d1
- net Net-(R67-Pad2) renamed /H_Bridge1/sw_o
- net Net-(R7-Pad1) renamed /H_Bridge2/d2
- net Net-(R80-Pad2) renamed /H_Bridge2/sw_o
- C22 pad 1: Net-(C22-Pad1) -> /H_Bridge0/sw_+
- C22 pad 2: Net-(C22-Pad2) -> /H_Bridge0/sw_s
- C23 pad 2: Net-(C23-Pad2) -> Net-(M2-ks)
- C24 pad 1: /H_Bridge0/-3.3 -> /H_Bridge0/0
- C64 pad 1: Net-(C64-Pad1) -> /H_Bridge1/sw_+
- C64 pad 2: Net-(C64-Pad2) -> /H_Bridge1/sw_s
- C65 pad 2: Net-(C65-Pad2) -> Net-(M4-ks)
- C66 pad 1: /H_Bridge1/-3.3 -> /H_Bridge1/0
- C74 pad 1: Net-(C74-Pad1) -> /H_Bridge2/sw_+
- C74 pad 2: Net-(C74-Pad2) -> /H_Bridge2/sw_s
- C75 pad 2: Net-(C75-Pad2) -> Net-(M6-ks)
- C76 pad 1: /H_Bridge2/-3.3 -> /H_Bridge2/0
- D3 pad A: /H_Bridge0/+12 -> Net-(D3-PadA)
- D3 pad C: Net-(D3-PadC) -> /H_Bridge0/sw_+
- D5 pad A: /H_Bridge1/+12 -> Net-(D5-PadA)
- D5 pad C: Net-(D5-PadC) -> /H_Bridge1/sw_+
- D7 pad A: /H_Bridge2/+12 -> Net-(D7-PadA)
- D7 pad C: Net-(D7-PadC) -> /H_Bridge2/sw_+
- HOLE3 pad 1: Net-(HOLE3-Pad1) -> unconnected-(HOLE3-Pad1)
- HOLE4 pad 1: Net-(HOLE4-Pad1) -> unconnected-(HOLE4-Pad1)
- J10 pad 1: /H_Bridge0/-3.3 -> /H_Bridge0/V_servo
- J10 pad 3: /H_Bridge0/C_N -> /H_Bridge0/C_P
- J10 pad 4: /H_Bridge0/C_P -> /H_Bridge0/C_N
- J11 pad 1: /H_Bridge1/-3.3 -> /H_Bridge1/V_servo
- J11 pad 3: /H_Bridge1/C_N -> /H_Bridge1/C_P
- J11 pad 4: /H_Bridge1/C_P -> /H_Bridge1/C_N
- J12 pad 1: /H_Bridge2/-3.3 -> /H_Bridge2/V_servo
- J12 pad 3: /H_Bridge2/C_N -> /H_Bridge2/C_P
- J12 pad 4: /H_Bridge2/C_P -> /H_Bridge2/C_N
- M1 pad KS: Net-(C25-Pad1) -> /H_Bridge0/sw_s
- M2 pad KS: Net-(C26-Pad1) -> Net-(M2-ks)
- M3 pad KS: Net-(C67-Pad1) -> /H_Bridge1/sw_s
- M4 pad KS: Net-(C68-Pad1) -> Net-(M4-ks)
- M5 pad KS: Net-(C77-Pad1) -> /H_Bridge2/sw_s
- M6 pad KS: Net-(C78-Pad1) -> Net-(M6-ks)
- R27 pad 1: Net-(C22-Pad1) -> /H_Bridge0/+12
- R27 pad 2: Net-(D3-PadC) -> Net-(D3-PadA)
- R33 pad 1: /H_Bridge0/I_P -> /H_Bridge0/I_N
- R33 pad 2: /H_Bridge0/I_N -> /H_Bridge0/I_P
- R34 pad 1: Net-(R34-Pad1) -> /H_Bridge0/C_N
- R34 pad 2: Net-(R34-Pad2) -> /H_Bridge0/C_P
- R34 pad 3: /H_Bridge0/I_N -> /H_Bridge0/I_P
- R34 pad 4: /H_Bridge0/I_P -> /H_Bridge0/I_N
- R65 pad 1: Net-(C64-Pad1) -> /H_Bridge1/+12
- R65 pad 2: Net-(D5-PadC) -> Net-(D5-PadA)
- R71 pad 1: /H_Bridge1/I_P -> /H_Bridge1/I_N
- R71 pad 2: /H_Bridge1/I_N -> /H_Bridge1/I_P
- R72 pad 1: Net-(R72-Pad1) -> /H_Bridge1/C_N
- R72 pad 2: Net-(R72-Pad2) -> /H_Bridge1/C_P
- R72 pad 3: /H_Bridge1/I_N -> /H_Bridge1/I_P
- R72 pad 4: /H_Bridge1/I_P -> /H_Bridge1/I_N
- R78 pad 1: Net-(C74-Pad1) -> /H_Bridge2/+12
- R78 pad 2: Net-(D7-PadC) -> Net-(D7-PadA)
- R84 pad 1: /H_Bridge2/I_P -> /H_Bridge2/I_N
- R84 pad 2: /H_Bridge2/I_N -> /H_Bridge2/I_P
- R85 pad 1: Net-(R85-Pad1) -> /H_Bridge2/C_N
- R85 pad 2: Net-(R85-Pad2) -> /H_Bridge2/C_P
- R85 pad 3: /H_Bridge2/I_N -> /H_Bridge2/I_P
- R85 pad 4: /H_Bridge2/I_P -> /H_Bridge2/I_N
- U1 pad 4: Net-(C22-Pad2) -> /H_Bridge0/sw_s
- U1 pad 6: Net-(C22-Pad1) -> /H_Bridge0/sw_+
- U2 pad 4: Net-(C23-Pad2) -> Net-(M2-ks)
- U3 pad 4: Net-(C64-Pad2) -> /H_Bridge1/sw_s
- U3 pad 6: Net-(C64-Pad1) -> /H_Bridge1/sw_+
- U4 pad 4: Net-(C65-Pad2) -> Net-(M4-ks)
- U5 pad 4: Net-(C74-Pad2) -> /H_Bridge2/sw_s
- U5 pad 6: Net-(C74-Pad1) -> /H_Bridge2/sw_+
- U6 pad 4: Net-(C75-Pad2) -> Net-(M6-ks)
Routing:
- net +797V: track 98.0 -> 0.00 mm
- net /H_Bridge1/sw_s: track 0.00 -> 39.6 mm
- net /H_Bridge0/sw_s: track 0.00 -> 39.6 mm
- net /H_Bridge2/sw_s: track 0.00 -> 39.6 mm
- net Net-(C74-Pad2): track 35.1 -> 0.00 mm
- net Net-(C64-Pad2): track 35.1 -> 0.00 mm
- net Net-(C22-Pad2): track 35.1 -> 0.00 mm
- net Net-(C25-Pad1): track 28.7 -> 0.00 mm
- net Net-(C77-Pad1): track 28.7 -> 0.00 mm
- net Net-(C67-Pad1): track 28.7 -> 0.00 mm
- net /H_Bridge1/V-: track 0.00 -> 22.1 mm
- net /H_Bridge0/V-: track 0.00 -> 22.1 mm
- net /H_Bridge2/+3.3: track 25.4 -> 7.53 mm
- net /H_Bridge1/+3.3: track 25.4 -> 7.82 mm
- net /H_Bridge0/+3.3: track 25.4 -> 7.82 mm
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- added copper zone on F.Cu, net /H_Bridge0/0
- added copper zone on F.Cu, net /H_Bridge1/0
- added copper zone on F.Cu, net /H_Bridge2/0

Commit message: Set the run bit in the timer for the POSIF.
Changed lines of the file:
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@@
     (fp_line (start 2.85 2.5) (end -2.85 2.5)
       (stroke (width 0.1) (type solid)) (layer "F.Fab"))
-    (pad "1" smd roundrect (at -2.55 0 180) (size 1.8 5.4) (layers "F.Cu" "F.Paste" "F.Mask") (roundrect_rratio 0.138889)
+    (pad "1" smd roundrect (at -2.55 0 180) (size 1.8 5.4) (layers "F.Cu" "F.Paste" "F.Mask") (roundrect_rratio 0.1388888889)
       (net 8 "+800V") (pintype "passive"))
-    (pad "2" smd roundrect (at 2.55 0 180) (size 1.8 5.4) (layers "F.Cu" "F.Paste" "F.Mask") (roundrect_rratio 0.138889)
+    (pad "2" smd roundrect (at 2.55 0 180) (size 1.8 5.4) (layers "F.Cu" "F.Paste" "F.Mask") (roundrect_rratio 0.1388888889)
       (net 54 "/H_Bridge0/V-") (pintype "passive"))
     (model "${KISYS3DMOD}/Capacitor_SMD.3dshapes/C_2220_5650Metric.wrl"
@@
     (fp_line (start 2.85 2.5) (end -2.85 2.5)
       (stroke (width 0.1) (type solid)) (layer "F.Fab"))
-    (pad "1" smd roundrect (at -2.55 0 180) (size 1.8 5.4) (layers "F.Cu" "F.Paste" "F.Mask") (roundrect_rratio 0.138889)
+    (pad "1" smd roundrect (at -2.55 0 180) (size 1.8 5.4) (layers "F.Cu" "F.Paste" "F.Mask") (roundrect_rratio 0.1388888889)
       (net 8 "+800V") (pintype "passive"))
-    (pad "2" smd roundrect (at 2.55 0 180) (size 1.8 5.4) (layers "F.Cu" "F.Paste" "F.Mask") (roundrect_rratio 0.138889)
+    (pad "2" smd roundrect (at 2.55 0 180) (size 1.8 5.4) (layers "F.Cu" "F.Paste" "F.Mask") (roundrect_rratio 0.1388888889)
       (net 55 "/H_Bridge1/V-") (pintype "passive"))
     (model "${KISYS3DMOD}/Capacitor_SMD.3dshapes/C_2220_5650Metric.wrl"
@@
     (fp_line (start 2.85 2.5) (end -2.85 2.5)
       (stroke (width 0.1) (type solid)) (layer "F.Fab"))
-    (pad "1" smd roundrect (at -2.55 0 180) (size 1.8 5.4) (layers "F.Cu" "F.Paste" "F.Mask") (roundrect_rratio 0.138889)
+    (pad "1" smd roundrect (at -2.55 0 180) (size 1.8 5.4) (layers "F.Cu" "F.Paste" "F.Mask") (roundrect_rratio 0.1388888889)
       (net 8 "+800V") (pintype "passive"))
-    (pad "2" smd roundrect (at 2.55 0 180) (size 1.8 5.4) (layers "F.Cu" "F.Paste" "F.Mask") (roundrect_rratio 0.138889)
+    (pad "2" smd roundrect (at 2.55 0 180) (size 1.8 5.4) (layers "F.Cu" "F.Paste" "F.Mask") (roundrect_rratio 0.1388888889)
       (net 56 "/H_Bridge2/V-") (pintype "passive"))
     (model "${KISYS3DMOD}/Capacitor_SMD.3dshapes/C_2220_5650Metric.wrl"
@@
     (fp_line (start 2.85 2.5) (end -2.85 2.5)
       (stroke (width 0.1) (type solid)) (layer "F.Fab"))
-    (pad "1" smd roundrect (at -2.55 0 90) (size 1.8 5.4) (layers "F.Cu" "F.Paste" "F.Mask") (roundrect_rratio 0.138889)
+    (pad "1" smd roundrect (at -2.55 0 90) (size 1.8 5.4) (layers "F.Cu" "F.Paste" "F.Mask") (roundrect_rratio 0.1388888889)
       (net 22 "/pe") (pintype "passive"))
-    (pad "2" smd roundrect (at 2.55 0 90) (size 1.8 5.4) (layers "F.Cu" "F.Paste" "F.Mask") (roundrect_rratio 0.138889)
+    (pad "2" smd roundrect (at 2.55 0 90) (size 1.8 5.4) (layers "F.Cu" "F.Paste" "F.Mask") (roundrect_rratio 0.1388888889)
       (net 56 "/H_Bridge2/V-") (pintype "passive"))
     (model "${KISYS3DMOD}/Capacitor_SMD.3dshapes/C_2220_5650Metric.wrl"
@@
     (fp_line (start 2.85 2.5) (end -2.85 2.5)
       (stroke (width 0.1) (type solid)) (layer "F.Fab"))
-    (pad "1" smd roundrect (at -2.55 0 90) (size 1.8 5.4) (layers "F.Cu" "F.Paste" "F.Mask") (roundrect_rratio 0.138889)
+    (pad "1" smd roundrect (at -2.55 0 90) (size 1.8 5.4) (layers "F.Cu" "F.Paste" "F.Mask") (roundrect_rratio 0.1388888889)
       (net 22 "/pe") (pintype "passive"))
-    (pad "2" smd roundrect (at 2.55 0 90) (size 1.8 5.4) (layers "F.Cu" "F.Paste" "F.Mask") (roundrect_rratio 0.138889)
+    (pad "2" smd roundrect (at 2.55 0 90) (size 1.8 5.4) (layers "F.Cu" "F.Paste" "F.Mask") (roundrect_rratio 0.1388888889)
       (net 8 "+800V") (pintype "passive"))
     (model "${KISYS3DMOD}/Capacitor_SMD.3dshapes/C_2220_5650Metric.wrl"
@@
     (fp_line (start 3.15 1.6) (end -3.15 1.6)
       (stroke (width 0.1) (type solid)) (layer "F.Fab"))
-    (pad "1" smd roundrect (at -2.9 0) (size 1.35 3.35) (layers "F.Cu" "F.Paste" "F.Mask") (roundrect_rratio 0.185185)
+    (pad "1" smd roundrect (at -2.9 0) (size 1.35 3.35) (layers "F.Cu" "F.Paste" "F.Mask") (roundrect_rratio 0.1851851852)
       (net 32 "/H_Bridge0/sw_m1") (pintype "passive"))
-    (pad "2" smd roundrect (at 2.9 0) (size 1.35 3.35) (layers "F.Cu" "F.Paste" "F.Mask") (roundrect_rratio 0.185185)
+    (pad "2" smd roundrect (at 2.9 0) (size 1.35 3.35) (layers "F.Cu" "F.Paste" "F.Mask") (roundrect_rratio 0.1851851852)
       (net 23 "/H_Bridge0/sw_m2") (pintype "passive"))
     (model "${KISYS3DMOD}/Resistor_SMD.3dshapes/R_2512_6332Metric.wrl"
@@
     (fp_line (start 3.15 1.6) (end -3.15 1.6)
       (stroke (width 0.1) (type solid)) (layer "F.Fab"))
-    (pad "1" smd roundrect (at -2.9 0) (size 1.35 3.35) (layers "F.Cu" "F.Paste" "F.Mask") (roundrect_rratio 0.185185)
+    (pad "1" smd roundrect (at -2.9 0) (size 1.35 3.35) (layers "F.Cu" "F.Paste" "F.Mask") (roundrect_rratio 0.1851851852)
       (net 33 "/H_Bridge1/sw_m1") (pintype "passive"))
-    (pad "2" smd roundrect (at 2.9 0) (size 1.35 3.35) (layers "F.Cu" "F.Paste" "F.Mask") (roundrect_rratio 0.185185)
+    (pad "2" smd roundrect (at 2.9 0) (size 1.35 3.35) (layers "F.Cu" "F.Paste" "F.Mask") (roundrect_rratio 0.1851851852)
       (net 24 "/H_Bridge1/sw_m2") (pintype "passive"))
     (model "${KISYS3DMOD}/Resistor_SMD.3dshapes/R_2512_6332Metric.wrl"
@@
     (fp_line (start 3.15 1.6) (end -3.15 1.6)
       (stroke (width 0.1) (type solid)) (layer "F.Fab"))
-    (pad "1" smd roundrect (at -2.9 0) (size 1.35 3.35) (layers "F.Cu" "F.Paste" "F.Mask") (roundrect_rratio 0.185185)
+    (pad "1" smd roundrect (at -2.9 0) (size 1.35 3.35) (layers "F.Cu" "F.Paste" "F.Mask") (roundrect_rratio 0.1851851852)
       (net 57 "/H_Bridge2/sw_m1") (pintype "passive"))
-    (pad "2" smd roundrect (at 2.9 0) (size 1.35 3.35) (layers "F.Cu" "F.Paste" "F.Mask") (roundrect_rratio 0.185185)
+    (pad "2" smd roundrect (at 2.9 0) (size 1.35 3.35) (layers "F.Cu" "F.Paste" "F.Mask") (roundrect_rratio 0.1851851852)
       (net 27 "/H_Bridge2/sw_m2") (pintype "passive"))
     (model "${KISYS3DMOD}/Resistor_SMD.3dshapes/R_2512_6332Metric.wrl"
