File: hv_control/hv_control.kicad_pcb (KiCad board)
At the start: 2 copper layers, 100 x 100 mm, 191 parts, among them J1 DB9, J10 x, J11 Conn_02x03_Odd_Even, J12 x, J13 Conn_01x02_Male, J14 Conn_01x02_Male, J15 Conn_01x02_Male, J16 Conn_01x02_Male, J17 Conn_01x02_Male, J2 DB15, J3 INPUTS, J4 I/O, J5 USB_B_Mini, J6 Conn_01x01_Male, J7 Conn_01x01_Male, J8 Conn_02x04_Odd_Even, J9 x, K1 RELAY_DPDT, K2 RELAY_DPDT, P2 SWD, P8 CONN_01X01, Q1 FOD817A300, Q2 BSS138, Q3 BSS138, U1 XMC4400-F100, U10 XMC1301T016F0032ABXUMA1, U11 LT1764EQ, U12 LMV331, U13 DRV8870DDA, U14 AD8226, U15 MAX3463, U18 LT1764EQ, U19 KSZ8081, U2 ips511g, U20 ETH100_MAG, U21 MAX3463, U22 MAX3463, U23 MAX3463, U3 ips511g, U30 FSL4110LR, U31 TL431MFDT, U4 MAX3463, U5 AD8226, U6 R-78E5.0-0.5, U7 TS321, U8 R-78E3.3-0.5, U9 ISO7321C, Y1 12MHz, Y2 25MHz

Commit message: Functional CRC
Routing:
- net GND: track 243.0 -> 237.2 mm

Commit message: Ordered new boards.
Parts:
- removed P8: CONN_01X01, Connector_PinHeader_2.54mm:PinHeader_1x01_P2.54mm_Vertical
- removed VR1, VR3: PEME1-S5-S3-S, 00_Passives:RKZXXXXS
- added C22: C, Capacitor_THT:C_Rect_L18.0mm_W6.0mm_P15.00mm_FKS3_FKP3, F.Cu at (156.8, 106.2)
- added C23: 100nF, Capacitor_SMD:C_0603_1608Metric, B.Cu at (92.8, 41.3)
- added C24: C, Capacitor_SMD:C_0603_1608Metric, B.Cu at (170.1, 96.5)
- added C25: 4.7uF, Capacitor_SMD:CP_Elec_10x14.3, F.Cu at (165.6, 103.0)
- added C63: 100nF, Capacitor_SMD:C_0603_1608Metric, F.Cu at (128.2, 81.8)
- added J18: Conn_01x01_Pin, Connector_Pin:Pin_D1.4mm_L8.5mm_W2.8mm_FlatFork, F.Cu at (156.8, 125.0)
- added J19: Conn_01x01_Pin, Connector_Pin:Pin_D1.4mm_L8.5mm_W2.8mm_FlatFork, F.Cu at (178.4, 78.8)
- added M1: Fan_4pin, Connector:FanPinHeader_1x04_P2.54mm_Vertical, F.Cu at (129.5, 54.6)
- added Q4: BSS138, Package_TO_SOT_SMD:SOT-23, F.Cu at (126.8, 79.0)
- added Q5: TCLT1003, Package_SO:SOP-4_3.8x7.5mm_P2.54mm, F.Cu at (132.0, 123.1)
- added R27: 27k, Resistor_SMD:R_0603_1608Metric, B.Cu at (162.1, 88.8)
- added R28: 3.3MEG, Resistor_SMD:R_1206_3216Metric, B.Cu at (170.5, 106.8)
- added R29: 3.3MEG, Resistor_SMD:R_1206_3216Metric, B.Cu at (170.5, 102.0)
- added R30: 27k, Resistor_SMD:R_0603_1608Metric, B.Cu at (171.6, 96.5)
- added R31: 120, Resistor_SMD:R_0603_1608Metric, B.Cu at (90.5, 42.0)
- added R32: 120, Resistor_SMD:R_0603_1608Metric, B.Cu at (99.7, 44.2)
- added R33: 62k, Resistor_SMD:R_0603_1608Metric, F.Cu at (118.0, 124.7)
- added R34: 1k, Resistor_SMD:R_0603_1608Metric, F.Cu at (117.8, 119.3)
- added R60: 1k, Resistor_SMD:R_0603_1608Metric, F.Cu at (126.5, 76.2)
- added R61: 0, Resistor_SMD:R_0805_2012Metric, F.Cu at (157.4, 55.4)
- added R62: 0, Resistor_SMD:R_0603_1608Metric, B.Cu at (99.5, 35.1)
- C2, C4: value 100uF/35V -> 100nF; footprint Capacitor_SMD:CP_Elec_8x10.5 -> Capacitor_SMD:C_0603_1608Metric; moved to B.Cu
- C48, C49: moved to F.Cu
- HOLE3, HOLE4: footprint MountingHole:MountingHole_3.2mm_M3 -> MountingHole:MountingHole_3.2mm_M3_DIN965_Pad
- J13, J14, J16, J17: footprint 00_Local:pin_2_5mm -> 00_Passives:pin_2_5mm
- J15: value Conn_01x02_Male -> Conn_01x01_Pin; footprint Connector_PinHeader_2.54mm:PinHeader_1x02_P2.54mm_Vertical -> Connector_Pin:Pin_D1.4mm_L8.5mm_W2.8mm_FlatFork
- J6: value Conn_01x01_Male -> Conn_01x01_Pin; footprint Connector_PinHeader_2.54mm:PinHeader_1x01_P2.54mm_Vertical -> Connector_Pin:Pin_D1.4mm_L8.5mm_W2.8mm_FlatFork
- K1, K2: footprint 00_Local:T77 -> 00_Passives:T77
- Q1: value FOD817A300 -> BSS138; footprint Package_DIP:DIP-4_W7.62mm -> Package_TO_SOT_SMD:SOT-23
- R100: value 4.7k -> 39k
- R15: value R -> 3.3MEG; footprint Resistor_SMD:R_0603_1608Metric -> Resistor_SMD:R_1206_3216Metric
- R16: value R -> 27k
- R88, R90: moved to B.Cu
- R97: value 150 -> 51
- R99: value 33k -> 91k
- U12: value LMV331 -> TLV9064; footprint Package_TO_SOT_SMD:SOT-23-5 -> Package_SO:SOIC-14_3.9x8.7mm_P1.27mm
- moved J6 89.5 mm to (170.5, 115.8), turned to 0 degrees
- moved C2 73.2 mm to (88.5, 94.2), turned to -90 degrees
- moved C4 64.7 mm to (88.5, 83.7), turned to -90 degrees
- moved C62 53.5 mm to (85.0, 110.0)
- moved U11 24.8 mm to (152.0, 89.0), turned to 0 degrees
- moved R15 23.4 mm to (170.5, 111.5), turned to -90 degrees
- moved J17 20.5 mm to (164.0, 39.8)
- moved J16 20.5 mm to (164.0, 60.2)
- moved C55 19.8 mm to (152.9, 96.2), turned to 180 degrees
- moved J15 16.5 mm to (151.2, 103.2)
- moved C34 14.5 mm to (163.0, 87.0), turned to -90 degrees
- moved C52 11.7 mm to (170.1, 93.5), turned to 90 degrees
- moved Q1 11.4 mm to (117.8, 122.0), turned to -90 degrees
- moved C39 10.0 mm to (90.5, 30.8)
- moved R88 9.12 mm to (151.7, 114.2), turned to 180 degrees
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Connections:
- net /ENC1_A/DATA renamed /ENC1_A/DATA
- net /ENC1_B/CLK renamed /ENC1_B/CLK
- net /ENC1_Z/SELECT renamed /ENC1_Z/SELECT
- net /ETH0_~RST renamed /ETH0_~{RST}
- net /Vfan renamed /Vmeas_24
- net /~A renamed /~{A}
- net /~B renamed /~{B}
- net /~Z renamed /~{Z}
- net Net-(C86-Pad1) renamed /flyback/VOLTAGE
- net Net-(J3-Pad1) renamed /AN_IN5
- net Net-(J3-Pad11) renamed /AN_IN0
- net Net-(J3-Pad3) renamed /AN_IN4
- net Net-(J3-Pad5) renamed /AN_IN3
- net Net-(J3-Pad7) renamed /AN_IN2
- net Net-(J3-Pad9) renamed /AN_IN1
- C2 pad 1: GNDPWR -> +5V
- C2 pad 2: -3.3Vp -> GND
- C4 pad 1: +800V -> +5V
- C4 pad 2: +797V -> GND
- C5 pad 1: Net-(C5-Pad1) -> Net-(U12B-+)
- C82 pad 1: Net-(C82-Pad1) -> Net-(Q5-C)
- D1 pad 2: /LED2 -> /LED1
- D1 pad 4: /LED0 -> /LED3
- D1 pad 6: /LED1 -> /LED2
- D1 pad 8: /LED3 -> /LED0
- HOLE2 pad 1: Net-(HOLE2-Pad1) -> unconnected-(HOLE2-Pad1)
- HOLE3 pad 1: Net-(HOLE3-Pad1) -> unconnected-(HOLE3-Pad1)
- J1 pad 16: (no net) -> Net-(HOLE1-Pad1)
- J10 pad 1: -3.3Vp -> unconnected-(J10-Pin_1-Pad1)
- J10 pad 3: /I1_N -> /I0_N
- J12 pad 1: -3.3Vp -> unconnected-(J12-Pin_1-Pad1)
- J12 pad 3: /I2_N -> /I0_N
- J15 pad 1: +797V -> +800V
- J16 pad 1: Net-(J16-Pad1) -> Net-(J16-Pin_1)
- J16 pad 2: GND -> Net-(J16-Pin_2)
- J17 pad 1: Net-(J17-Pad1) -> GND
- J2 pad 16: (no net) -> Net-(HOLE4-Pad1)
- J6 pad 1: /TRACESWO -> Net-(J6-Pin_1)
- J9 pad 1: -3.3Vp -> unconnected-(J9-Pin_1-Pad1)
- Q1 pad 1: +12V -> /SUPPLY_VOLTAGE
- Q1 pad 2: Net-(Q1-Pad2) -> GND
- Q1 pad 3: Net-(C82-Pad1) -> Net-(Q1-D)
- R13 pad 1: Net-(R13-Pad1) -> Net-(U12B-+)
- R14 pad 1: Net-(R13-Pad1) -> Net-(U12B-+)
- R15 pad 2: Net-(C5-Pad1) -> Net-(J6-Pin_1)
- R16 pad 1: +3.3VP -> Net-(U12C-+)
- R16 pad 2: Net-(R16-Pad2) -> +3.3VP
- R2 pad 1: /LED0 -> /LED3
- R2 pad 2: /TRACED1 -> /TRACED3
- R3 pad 1: /LED1 -> /LED2
- R4 pad 1: /LED2 -> /LED1
- R4 pad 2: /TRACED3 -> /TRACED1
- R5 pad 1: /LED3 -> /LED0
- R93 pad 1: Net-(C82-Pad1) -> Net-(Q5-C)
- R94 pad 1: Net-(Q1-Pad2) -> Net-(Q5-k)
- R95 pad 2: Net-(Q1-Pad2) -> Net-(Q5-k)
- U1 pad 13: Net-(U1-Pad13) -> unconnected-(U1A-HIB_IO_1-Pad13)
- U1 pad 14: Net-(U1-Pad14) -> unconnected-(U1A-HIB_IO_0-Pad14)
- U1 pad 15: Net-(U1-Pad15) -> unconnected-(U1A-RTC_XTAL1-Pad15)
- U1 pad 16: Net-(U1-Pad16) -> unconnected-(U1A-RTC_XTAL2-Pad16)
- U1 pad 18: Net-(U1-Pad18) -> unconnected-(U1A-P15.3-Pad18)
- U1 pad 19: Net-(U1-Pad19) -> unconnected-(U1A-P15.2-Pad19)
- U1 pad 20: Net-(U1-Pad20) -> /ENC_REF
- U1 pad 3: Net-(U1-Pad3) -> /COPRO_POWER
- U1 pad 4: /PWM0 -> /SUPPLY_VOLTAGE
- U1 pad 50: Net-(U1-Pad50) -> unconnected-(U1B-P2.2-Pad50)
- U1 pad 69: Net-(U1-Pad69) -> unconnected-(U1C-P1.14-Pad69)
- U1 pad 70: Net-(U1-Pad70) -> /IO0
- U1 pad 72: Net-(U1-Pad72) -> /ENC0_CDIR
- U1 pad 78: /IO0 -> /ENC0_CLK
- U1 pad 83: Net-(U1-Pad83) -> /IO5
- U1 pad 91: /IO5 -> /IO6
- U1 pad 92: /IO6 -> /IO7
- U1 pad 93: /IO7 -> /PWM0
- U1 pad 94: Net-(U1-Pad94) -> /fan
- U10 pad 10: Net-(U10-Pad10) -> unconnected-(U10-P0.7-Pad10)
- U10 pad 11: Net-(U10-Pad11) -> unconnected-(U10-P0.8-Pad11)
- U10 pad 12: Net-(U10-Pad12) -> unconnected-(U10-P0.9-Pad12)
- U10 pad 16: /I0_N -> unconnected-(U10-P2.6-Pad16)
- U10 pad 2: /I2_N -> Net-(U10-P2.9)
- U10 pad 3: /I1_N -> Net-(U10-P2.10)
- U10 pad 7: Net-(R15-Pad1) -> unconnected-(U10-P0.0-Pad7)
- U10 pad 8: Net-(R16-Pad2) -> unconnected-(U10-P0.5-Pad8)
- U10 pad 9: Net-(U10-Pad9) -> unconnected-(U10-P0.6-Pad9)
- U12 pad 1: Net-(R13-Pad1) -> Net-(U10-P2.9)
- U12 pad 2: GNDPWR -> Net-(U10-P2.9)
- U12 pad 3: Net-(C5-Pad1) -> Net-(U12A-+)
- U12 pad 4: Net-(R16-Pad2) -> +3.3VP
- U12 pad 5: +3.3VP -> Net-(U12B-+)
- U13 pad 6: Net-(J16-Pad1) -> Net-(J16-Pin_2)
- U13 pad 8: Net-(J17-Pad1) -> Net-(J16-Pin_1)
- U14 pad 6: Net-(U14-Pad6) -> /ENC_REF
- U15 pad 2: GND -> /ENC0_CDIR
- U15 pad 3: GND -> /ENC0_CDIR
- U15 pad 4: GND -> /ENC0_CLK
- U19 pad 18: Net-(U19-Pad18) -> unconnected-(U19-INTRP-Pad18)
- U30 pad 3: Net-(C82-Pad1) -> Net-(Q5-C)
- U5 pad 6: Net-(U14-Pad6) -> /ENC_REF
- U7 pad 1: Net-(U14-Pad6) -> /ENC_REF
- U7 pad 4: Net-(U14-Pad6) -> /ENC_REF
- VR2 pad 2: GND -> Net-(Q4-D)
- Y1 pad 2: Net-(Y1-Pad2) -> GND
- Y1 pad 4: Net-(Y1-Pad4) -> GND
- Y2 pad 2: Net-(Y2-Pad2) -> GND
- Y2 pad 4: Net-(Y2-Pad4) -> GND
Routing:
- net GNDPWR: track 273.4 -> 125.1 mm, vias 2 -> 13
- net -3.3Vp: track 117.3 -> 0.00 mm, vias 3 -> 0
- net /SUPPLY_VOLTAGE: track 0.00 -> 82.2 mm, vias 0 -> 1
- net /ENC_REF: track 0.00 -> 57.5 mm, vias 0 -> 2
- net GND: track 237.2 -> 182.5 mm, vias 60 -> 68
- net /I0_N: track 30.3 -> 84.6 mm, vias 0 -> 2
- net +797V: track 41.9 -> 0.00 mm
- net /COPRO_POWER: track 0.00 -> 35.8 mm, vias 0 -> 1
- net Net-(J16-Pad1): track 34.5 -> 0.00 mm
- net /ENC0_CLK: track 0.00 -> 33.8 mm, vias 0 -> 2
- net /I2_N: track 31.4 -> 0.00 mm
- net /ENC0_CDIR: track 0.00 -> 27.4 mm
- net Net-(U14-Pad6): track 27.1 -> 0.00 mm
- net +3.3VADC: track 60.7 -> 87.2 mm
- net +12V: track 318.8 -> 296.3 mm
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- added copper zone on F.Cu, net GNDPWR
Other:
- board text added: "hv_control 2.0"

Commit message: Set the run bit in the timer for the POSIF.
Changed lines of the file:
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@@
     (aux_axis_origin 80.5 127.5)
     (pcbplotparams
-      (layerselection 0x00010fc_ffffffff)
+      (layerselection 0x00010ec_ffffffff)
       (plot_on_all_layers_selection 0x0000000_00000000)
       (disableapertmacros false)
@@
     (fp_line (start 1 0.625) (end -1 0.625)
       (stroke (width 0.1) (type solid)) (layer "F.Fab"))
-    (pad "1" smd roundrect (at -0.9125 0 270) (size 1.025 1.4) (layers "F.Cu" "F.Paste" "F.Mask") (roundrect_rratio 0.243902)
+    (pad "1" smd roundrect (at -0.9125 0 270) (size 1.025 1.4) (layers "F.Cu" "F.Paste" "F.Mask") (roundrect_rratio 0.243902439)
       (net 1 "+12V") (pintype "passive"))
-    (pad "2" smd roundrect (at 0.9125 0 270) (size 1.025 1.4) (layers "F.Cu" "F.Paste" "F.Mask") (roundrect_rratio 0.243902)
+    (pad "2" smd roundrect (at 0.9125 0 270) (size 1.025 1.4) (layers "F.Cu" "F.Paste" "F.Mask") (roundrect_rratio 0.243902439)
       (net 162 "+24V") (pintype "passive"))
     (model "${KICAD6_3DMODEL_DIR}/Resistor_SMD.3dshapes/R_0805_2012Metric.wrl"
@@
     (fp_line (start 2 2) (end 2 -2)
       (stroke (width 0.1) (type solid)) (layer "B.Fab"))
-    (pad "" smd roundrect (at -0.65 -0.65 90) (size 1.05 1.05) (layers "B.Paste") (roundrect_rratio 0.238095))
-    (pad "" smd roundrect (at -0.65 0.65 90) (size 1.05 1.05) (layers "B.Paste") (roundrect_rratio 0.238095))
-    (pad "" smd roundrect (at 0.65 -0.65 90) (size 1.05 1.05) (layers "B.Paste") (roundrect_rratio 0.238095))
-    (pad "" smd roundrect (at 0.65 0.65 90) (size 1.05 1.05) (layers "B.Paste") (roundrect_rratio 0.238095))
+    (pad "" smd roundrect (at -0.65 -0.65 90) (size 1.05 1.05) (layers "B.Paste") (roundrect_rratio 0.2380952381))
+    (pad "" smd roundrect (at -0.65 0.65 90) (size 1.05 1.05) (layers "B.Paste") (roundrect_rratio 0.2380952381))
+    (pad "" smd roundrect (at 0.65 -0.65 90) (size 1.05 1.05) (layers "B.Paste") (roundrect_rratio 0.2380952381))
+    (pad "" smd roundrect (at 0.65 0.65 90) (size 1.05 1.05) (layers "B.Paste") (roundrect_rratio 0.2380952381))
     (pad "1" smd roundrect (at -1.9375 1.25 90) (size 0.825 0.25) (layers "B.Cu" "B.Paste" "B.Mask") (roundrect_rratio 0.25)
       (net 15 "Net-(U19-Vdd_1.2)") (pinfunction "Vdd_1.2") (pintype "input"))
@@
     (pad "24" smd roundrect (at -1.25 1.9375 90) (size 0.25 0.825) (layers "B.Cu" "B.Paste" "B.Mask") (roundrect_rratio 0.25)
       (net 47 "/ETH0_~{RST}") (pinfunction "~{RST}") (pintype "input"))
-    (pad "25" smd roundrect (at 0 0 90) (size 2.6 2.6) (layers "B.Cu" "B.Mask") (roundrect_rratio 0.096154)
+    (pad "25" smd roundrect (at 0 0 90) (size 2.6 2.6) (layers "B.Cu" "B.Mask") (roundrect_rratio 0.09615384615)
       (net 2 "GND") (pinfunction "GND") (pintype "input"))
     (model "${KISYS3DMOD}/Package_DFN_QFN.3dshapes/QFN-24-1EP_4x4mm_P0.5mm_EP2.6x2.6mm.wrl"
@@
     (fp_line (start 2.5 1.25) (end 2.5 -1.25)
       (stroke (width 0.1) (type solid)) (layer "B.Fab"))
-    (pad "1" smd roundrect (at -2.25 0 270) (size 1.35 2.65) (layers "B.Cu" "B.Paste" "B.Mask") (roundrect_rratio 0.185185)
+    (pad "1" smd roundrect (at -2.25 0 270) (size 1.35 2.65) (layers "B.Cu" "B.Paste" "B.Mask") (roundrect_rratio 0.1851851852)
       (net 91 "Net-(C83-Pad1)") (pintype "passive"))
-    (pad "2" smd roundrect (at 2.25 0 270) (size 1.35 2.65) (layers "B.Cu" "B.Paste" "B.Mask") (roundrect_rratio 0.185185)
+    (pad "2" smd roundrect (at 2.25 0 270) (size 1.35 2.65) (layers "B.Cu" "B.Paste" "B.Mask") (roundrect_rratio 0.1851851852)
       (net 90 "/flyback/sw") (pintype "passive"))
     (model "${KISYS3DMOD}/Resistor_SMD.3dshapes/R_2010_5025Metric.wrl"
@@
     (fp_line (start 1.6 0.8) (end 1.6 -0.8)
       (stroke (width 0.1) (type solid)) (layer "B.Fab"))
-    (pad "1" smd roundrect (at -1.4625 0 270) (size 1.125 1.75) (layers "B.Cu" "B.Paste" "B.Mask") (roundrect_rratio 0.222222)
+    (pad "1" smd roundrect (at -1.4625 0 270) (size 1.125 1.75) (layers "B.Cu" "B.Paste" "B.Mask") (roundrect_rratio 0.2222222222)
       (net 179 "Net-(R28-Pad1)") (pintype "passive"))
-    (pad "2" smd roundrect (at 1.4625 0 270) (size 1.125 1.75) (layers "B.Cu" "B.Paste" "B.Mask") (roundrect_rratio 0.222222)
+    (pad "2" smd roundrect (at 1.4625 0 270) (size 1.125 1.75) (layers "B.Cu" "B.Paste" "B.Mask") (roundrect_rratio 0.2222222222)
       (net 177 "Net-(R15-Pad1)") (pintype "passive"))
     (model "${KICAD6_3DMODEL_DIR}/Resistor_SMD.3dshapes/R_1206_3216Metric.wrl"
@@
     (fp_line (start 1.6 0.8) (end 1.6 -0.8)
       (stroke (width 0.1) (type solid)) (layer "B.Fab"))
-    (pad "1" smd roundrect (at -1.4625 0 270) (size 1.125 1.75) (layers "B.Cu" "B.Paste" "B.Mask") (roundrect_rratio 0.222222)
+    (pad "1" smd roundrect (at -1.4625 0 270) (size 1.125 1.75) (layers "B.Cu" "B.Paste" "B.Mask") (roundrect_rratio 0.2222222222)
       (net 176 "Net-(U12A-+)") (pintype "passive"))
-    (pad "2" smd roundrect (at 1.4625 0 270) (size 1.125 1.75) (layers "B.Cu" "B.Paste" "B.Mask") (roundrect_rratio 0.222222)
+    (pad "2" smd roundrect (at 1.4625 0 270) (size 1.125 1.75) (layers "B.Cu" "B.Paste" "B.Mask") (roundrect_rratio 0.2222222222)
       (net 179 "Net-(R28-Pad1)") (pintype "passive"))
     (model "${KICAD6_3DMODEL_DIR}/Resistor_SMD.3dshapes/R_1206_3216Metric.wrl"
@@
     (fp_line (start 1.6 0.8) (end 1.6 -0.8)
       (stroke (width 0.1) (type solid)) (layer "B.Fab"))
-    (pad "1" smd roundrect (at -1.4625 0 270) (size 1.125 1.75) (layers "B.Cu" "B.Paste" "B.Mask") (roundrect_rratio 0.222222)
+    (pad "1" smd roundrect (at -1.4625 0 270) (size 1.125 1.75) (layers "B.Cu" "B.Paste" "B.Mask") (roundrect_rratio 0.2222222222)
       (net 177 "Net-(R15-Pad1)") (pintype "passive"))
-    (pad "2" smd roundrect (at 1.4625 0 270) (size 1.125 1.75) (layers "B.Cu" "B.Paste" "B.Mask") (roundrect_rratio 0.222222)
+    (pad "2" smd roundrect (at 1.4625 0 270) (size 1.125 1.75) (layers "B.Cu" "B.Paste" "B.Mask") (roundrect_rratio 0.2222222222)
       (net 184 "Net-(J6-Pin_1)") (pintype "passive"))
     (model "${KICAD6_3DMODEL_DIR}/Resistor_SMD.3dshapes/R_1206_3216Metric.wrl"

Commit message: Backup
Parts:
- C24, C5: value C -> 10nF
- C85, C90, C91: value 22uF/100V -> 100uF/35V
- R47, R48: value 10k -> 27k
- R90: value 100k -> 0
- U20: value ETH100_MAG -> SI-50170-F
