File: hv_control/hv_control.kicad_sch (KiCad schematic)
At the start: 176 parts, among them J1 DB9, J10 x, J11 Conn_02x03_Odd_Even, J12 x, J13 Conn_01x02_Male, J14 Conn_01x02_Male, J15 Conn_01x01_Pin, J16 Conn_01x02_Male, J17 Conn_01x02_Male, J18 Conn_01x01_Pin, J19 Conn_01x01_Pin, J2 DB15, J3 INPUTS, J4 I/O, J5 USB_B_Mini, J6 Conn_01x01_Pin, J7 Conn_01x01_Male, J8 Conn_02x04_Odd_Even, J9 x, K1 RELAY_DPDT, K2 RELAY_DPDT, M1 Fan_4pin, P2 SWD, Q1 BSS138, Q2 BSS138, Q3 BSS138, Q4 BSS138, U1 XMC4400-F100, U10 XMC1301T016F0032ABXUMA1, U11 LT1764EQ, U12 TLV9064, U13 DRV8870DDA, U14 AD8226, U15 MAX3463, U18 LT1764EQ, U19 KSZ8081, U2 ips511g, U20 SI-50170-F, U21 MAX3463, U22 MAX3463, U23 MAX3463, U3 ips511g, U4 MAX3463, U5 AD8226, U6 R-78E5.0-0.5, U7 ${SIM.PARAMS}, U8 R-78E3.3-0.5, U9 ISO7321C, Y1 12MHz, Y2 25MHz

Commit message: Comments for next version added.
Other:
- note added: "FIXME Opto pinning RXD_TIMER on P0.9 of XMC1301 100nF parallel with R27 (ook gnd beter aansluiten) Gaten sub-d te klein Opto geisoleerde ingangen op XH connector toevoegen"
- note removed: "FIXME Opto pinning RXD_TIMER on P0.9 of XMC1301 100nF parallel with R27 Gaten sub-d te klein"
Changed lines of the file:
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@@
     (effects (font (size 1.27 1.27)) (justify left bottom))
   )
-  (text "FIXME\n\nOpto pinning\nRXD_TIMER on P0.9 of XMC1301\n100nF parallel with R27\nGaten sub-d te klein"
+  (text "FIXME\n\nOpto pinning\nRXD_TIMER on P0.9 of XMC1301\n100nF parallel with R27 (ook gnd beter aansluiten)\nGaten sub-d te klein\nOpto geisoleerde ingangen op XH connector toevoegen"
     (at 322.58 36.83 0)
     (effects (font (size 1.27 1.27)) (justify left bottom))

Commit message: Comments for next hardware version.
Other:
- note added: "FIXME Opto pinning RXD_TIMER on P0.9 of XMC1301 100nF parallel with R27 (ook gnd beter aansluiten) Gaten sub-d te klein Opto geisoleerde ingangen op XH connector toevoegen Pin-4 of sub-d 9 is shield."
- note removed: "FIXME Opto pinning RXD_TIMER on P0.9 of XMC1301 100nF parallel with R27 (ook gnd beter aansluiten) Gaten sub-d te klein Opto geisoleerde ingangen op XH connector toevoegen"
Changed lines of the file:
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@@
     (effects (font (size 1.27 1.27)) (justify left bottom))
   )
-  (text "FIXME\n\nOpto pinning\nRXD_TIMER on P0.9 of XMC1301\n100nF parallel with R27 (ook gnd beter aansluiten)\nGaten sub-d te klein\nOpto geisoleerde ingangen op XH connector toevoegen"
+  (text "FIXME\n\nOpto pinning\nRXD_TIMER on P0.9 of XMC1301\n100nF parallel with R27 (ook gnd beter aansluiten)\nGaten sub-d te klein\nOpto geisoleerde ingangen op XH connector toevoegen\nPin-4 of sub-d 9 is shield."
     (at 322.58 36.83 0)
     (effects (font (size 1.27 1.27)) (justify left bottom))

Commit message: Backup
Other:
- note added: "FIXME Opto pinning RXD_TIMER on P0.9 of XMC1301 100nF parallel with R27 (ook gnd beter aansluiten) Gaten sub-d te klein Opto geisoleerde ingangen op XH connector toevoegen Pin-4 of sub-d 9 is shield. Signalen lineaal 1k // 330pF naar gnd Bredere digitale isolator Grotere gaten dc-dc converter"
- note removed: "FIXME Opto pinning RXD_TIMER on P0.9 of XMC1301 100nF parallel with R27 (ook gnd beter aansluiten) Gaten sub-d te klein Opto geisoleerde ingangen op XH connector toevoegen Pin-4 of sub-d 9 is shield."
